File: BenchBudEE/Power.sch (KiCad schematic (older format))
At the start: 14 parts

Commit message: checking in all my local changes before syncing to chris's repo.
Parts:
- gave numbers to parts that had none: 14
Changed lines of the file:
@@
 Sheet 4 9
 Title ""
-Date "24 feb 2014"
+Date "2 mar 2014"
 Rev ""
 Comp ""
@@
 $EndDescr
 $Comp
-L 5566-20A C?
+L 5566-20A C1
 U 1 1 52FAEACC
 P 3850 3750
-F 0 "C?" H 3500 4300 60  0000 C CNN
+F 0 "C1" H 3500 4300 60  0000 C CNN
 F 1 "5566-20A" H 4000 3200 60  0000 C CNN
 F 2 "~" H 3850 3750 60  0000 C CNN
@@
 $EndComp
 $Comp
-L +3.3V #PWR?
+L +3.3V #PWR14
 U 1 1 52FAEADB
 P 4650 3000
-F 0 "#PWR?" H 4650 2960 30  0001 C CNN
+F 0 "#PWR14" H 4650 2960 30  0001 C CNN
 F 1 "+3.3V" H 4650 3110 30  0000 C CNN
 F 2 "" H 4650 3000 60  0000 C CNN
@@
 $EndComp
 $Comp
-L GND #PWR?
+L GND #PWR13
 U 1 1 52FAEB0C
 P 3050 4300
-F 0 "#PWR?" H 3050 4300 30  0001 C CNN
+F 0 "#PWR13" H 3050 4300 30  0001 C CNN
 F 1 "GND" H 3050 4230 30  0001 C CNN
 F 2 "" H 3050 4300 60  0000 C CNN
@@
 $EndComp
 $Comp
-L GND #PWR?
+L GND #PWR15
 U 1 1 52FAEB39
 P 4650 4300
-F 0 "#PWR?" H 4650 4300 30  0001 C CNN
+F 0 "#PWR15" H 4650 4300 30  0001 C CNN
 F 1 "GND" H 4650 4230 30  0001 C CNN
 F 2 "" H 4650 4300 60  0000 C CNN
@@
 $EndComp
 $Comp
-L +5V #PWR?
+L +5V #PWR12
 U 1 1 52FAEB81
 P 2950 3500
-F 0 "#PWR?" H 2950 3590 20  0001 C CNN
+F 0 "#PWR12" H 2950 3590 20  0001 C CNN
 F 1 "+5V" H 2950 3590 30  0000 C CNN
 F 2 "" H 2950 3500 60  0000 C CNN
@@
 $EndComp
 $Comp
-L -12V #PWR?
+L -12V #PWR16
 U 1 1 52FAED85
 P 4850 3400
-F 0 "#PWR?" H 4850 3530 20  0001 C CNN
+F 0 "#PWR16" H 4850 3530 20  0001 C CNN
 F 1 "-12V" H 4850 3500 30  0000 C CNN
 F 2 "" H 4850 3400 60  0000 C CNN
@@
 $EndComp
 $Comp
-L -5V #PWR?
+L -5V #PWR17
 U 1 1 52FAEDD1
 P 4850 4100
-F 0 "#PWR?" H 4850 4240 20  0001 C CNN
+F 0 "#PWR17" H 4850 4240 20  0001 C CNN
 F 1 "-5V" H 4850 4210 30  0000 C CNN
 F 2 "" H 4850 4100 60  0000 C CNN
@@
 $EndComp
 $Comp
-L +12V #PWR?
+L +12V #PWR11
 U 1 1 52FAEE51
 P 2850 4100
-F 0 "#PWR?" H 2850 4050 20  0001 C CNN
+F 0 "#PWR11" H 2850 4050 20  0001 C CNN
 F 1 "+12V" H 2850 4200 30  0000 C CNN
 F 2 "" H 2850 4100 60  0000 C CNN
@@
 $EndComp
 $Comp
-L SWITCH_INV SW?
+L SWITCH_INV SW1
 U 1 1 52FAF3C7
 P 5850 3100
-F 0 "SW?" H 5650 3250 50  0000 C CNN
+F 0 "SW1" H 5650 3250 50  0000 C CNN
 F 1 "SWITCH_INV" H 5700 2950 50  0000 C CNN
 F 2 "~" H 5850 3100 60  0000 C CNN
@@
 $EndComp
 $Comp
-L GND #PWR?
+L GND #PWR18
 U 1 1 52FAED7C
 P 6450 3300
-F 0 "#PWR?" H 6450 3300 30  0001 C CNN
+F 0 "#PWR18" H 6450 3300 30  0001 C CNN
 F 1 "GND" H 6450 3230 30  0001 C CNN
 F 2 "" H 6450 3300 60  0000 C CNN
@@
 $EndComp
 $Comp
-L R R?
+L R R13
 U 1 1 52FAEDB5
 P 5000 3100
-F 0 "R?" V 5080 3100 40  0000 C CNN
+F 0 "R13" V 5080 3100 40  0000 C CNN
 F 1 "R" V 5007 3101 40  0000 C CNN
 F 2 "~" V 4930 3100 30  0000 C CNN
@@
 $EndComp
 $Comp
-L INDUCTOR L?
+L INDUCTOR L1
 U 1 1 52FAEFE1
 P 9250 3100
-F 0 "L?" V 9200 3100 40  0000 C CNN
+F 0 "L1" V 9200 3100 40  0000 C CNN
 F 1 "INDUCTOR" V 9350 3100 40  0000 C CNN
 F 2 "~" H 9250 3100 60  0000 C CNN
@@
 $EndComp
 $Comp
-L INDUCTOR L?
+L INDUCTOR L2
 U 1 1 52FAEFF6
 P 9250 4300
-F 0 "L?" V 9200 4300 40  0000 C CNN
+F 0 "L2" V 9200 4300 40  0000 C CNN
 F 1 "INDUCTOR" V 9350 4300 40  0000 C CNN
 F 2 "~" H 9250 4300 60  0000 C CNN
@@
 $EndComp
 $Comp
-L GND #PWR?
+L GND #PWR19
 U 1 1 52FAF0CD
 P 9950 3800
-F 0 "#PWR?" H 9950 3800 30  0001 C CNN
+F 0 "#PWR19" H 9950 3800 30  0001 C CNN
 F 1 "GND" H 9950 3730 30  0001 C CNN
 F 2 "" H 9950 3800 60  0000 C CNN
@@
 $EndComp
 $Comp
-L CP1 C?
+L CP1 C2
 U 1 1 52FAF15D
 P 9650 3400
-F 0 "C?" H 9700 3500 50  0000 L CNN
+F 0 "C2" H 9700 3500 50  0000 L CNN
 F 1 "CP1" H 9700 3300 50  0000 L CNN
 F 2 "~" H 9650 3400 60  0000 C CNN
@@
 $EndComp
 $Comp
-L CP1 C?
+L CP1 C3
 U 1 1 52FAF16A
 P 9650 4000
-F 0 "C?" H 9700 4100 50  0000 L CNN
+F 0 "C3" H 9700 4100 50  0000 L CNN
 F 1 "CP1" H 9700 3900 50  0000 L CNN
 F 2 "~" H 9650 4000 60  0000 C CNN
@@
 $EndComp
 $Comp
-L R R?
+L R R15
 U 1 1 52FAF170
 P 8600 4300
-F 0 "R?" V 8680 4300 40  0000 C CNN
+F 0 "R15" V 8680 4300 40  0000 C CNN
 F 1 "R" V 8607 4301 40  0000 C CNN
 F 2 "~" V 8530 4300 30  0000 C CNN
@@
 $EndComp
 $Comp
-L R R?
+L R R14
 U 1 1 52FAF176
 P 8600 3100
-F 0 "R?" V 8680 3100 40  0000 C CNN
+F 0 "R14" V 8680 3100 40  0000 C CNN
 F 1 "R" V 8607 3101 40  0000 C CNN
 F 2 "~" V 8530 3100 30  0000 C CNN
@@
 -12V_FILTERED
 $Comp
-L THERMISTOR TH?
+L THERMISTOR TH3
 U 1 1 53094891
 P 2600 3600
-F 0 "TH?" V 2700 3650 50  0000 C CNN
+F 0 "TH3" V 2700 3650 50  0000 C CNN
 F 1 "THERMISTOR" V 2500 3600 50  0000 C CNN
 F 2 "~" H 2600 3600 60  0000 C CNN
@@
 $EndComp
 $Comp
-L THERMISTOR TH?
+L THERMISTOR TH1
 U 1 1 530948AA
 P 2300 4200
-F 0 "TH?" V 2400 4250 50  0000 C CNN
+F 0 "TH1" V 2400 4250 50  0000 C CNN
 F 1 "THERMISTOR" V 2200 4200 50  0000 C CNN
 F 2 "~" H 2300 4200 60  0000 C CNN
@@
 $EndComp
 $Comp
-L THERMISTOR TH?
+L THERMISTOR TH2
 U 1 1 530949A6
 P 2600 3100
-F 0 "TH?" V 2700 3150 50  0000 C CNN
+F 0 "TH2" V 2700 3150 50  0000 C CNN
 F 1 "THERMISTOR" V 2500 3100 50  0000 C CNN
 F 2 "~" H 2600 3100 60  0000 C CNN
@@
 $EndComp
 $Comp
-L THERMISTOR TH?
+L THERMISTOR TH4
 U 1 1 530949B5
 P 5200 3400
-F 0 "TH?" V 5300 3450 50  0000 C CNN
+F 0 "TH4" V 5300 3450 50  0000 C CNN
 F 1 "THERMISTOR" V 5100 3400 50  0000 C CNN
 F 2 "~" H 5200 3400 60  0000 C CNN
@@
 $EndComp
 $Comp
-L THERMISTOR TH?
+L THERMISTOR TH5
 U 1 1 530949C4
 P 5200 4000
-F 0 "TH?" V 5300 4050 50  0000 C CNN
+F 0 "TH5" V 5300 4050 50  0000 C CNN
 F 1 "THERMISTOR" V 5100 4000 50  0000 C CNN
 F 2 "~" H 5200 4000 60  0000 C CNN
