File: BenchBudEE/Power.sch (KiCad schematic (older format))
At the start: 14 parts

Commit message: syncing to https://github.com/ContextualElectronics/BenchBudEE/tree/ebd662c68b928f78643cdf924dc35a4d91f03121
Parts:
- removed C?: 5566-20A, ~, symbol 5566-20A
- removed C? (x2): CP1, ~, symbol CP1
- removed L? (x2): INDUCTOR, ~, symbol INDUCTOR
- removed R? (x3): R, ~, symbol R
- removed SW?: SWITCH_INV, ~, symbol SWITCH_INV
- removed TH? (x5): THERMISTOR, ~, symbol THERMISTOR
- added C? (x3): C, ~, symbol C
- added L? (x3): INDUCTOR, ~, symbol INDUCTOR
- added P?: CONN_12X2, symbol CONN_12X2
- added R?: R, ~, symbol R
- added SW?: SWITCH_INV, ~, symbol SWITCH_INV
- added TH? (x4): THERMISTOR, ~, symbol THERMISTOR
Connections:
- net labels added: +12C, +12P, +3.3VP, +5P, -12P
- net labels removed: -12V_FILTERED, -12V_FUSED, -5V, -5V_FUSED, 12V_FILTERED, 12V_FUSED, 3.3V_FUSED, 5V_FUSED
- wire segments 58 -> 55

Commit message: playing with the layout
Parts:
- gave numbers to parts that had none: 13
Changed lines of the file:
@@
-EESchema Schematic File Version 2  date 10/10/2013 12:18:22 AM
+EESchema Schematic File Version 2
 LIBS:power
 LIBS:device
@@
 Sheet 3 9
 Title ""
-Date "10 oct 2013"
+Date "3 mar 2014"
 Rev ""
 Comp ""
@@
 $EndDescr
 $Comp
-L CONN_12X2 P?
+L CONN_12X2 P301
 U 1 1 523DFA5D
 P 2650 2050
-F 0 "P?" H 2650 2700 60  0000 C CNN
+F 0 "P301" H 2650 2700 60  0000 C CNN
 F 1 "CONN_12X2" V 2650 2050 50  0000 C CNN
 F 2 "" H 2650 2050 60  0000 C CNN
@@
 $EndComp
 $Comp
-L GND #PWR?
+L GND #PWR011
 U 1 1 523DFA76
 P 1400 1850
-F 0 "#PWR?" H 1400 1850 30  0001 C CNN
+F 0 "#PWR011" H 1400 1850 30  0001 C CNN
 F 1 "GND" H 1400 1780 30  0001 C CNN
 F 2 "" H 1400 1850 60  0000 C CNN
@@
 $EndComp
 $Comp
-L SWITCH_INV SW?
+L SWITCH_INV SW301
 U 1 1 523DFB25
 P 4100 3100
-F 0 "SW?" H 3900 3250 50  0000 C CNN
+F 0 "SW301" H 3900 3250 50  0000 C CNN
 F 1 "SWITCH_INV" H 3950 2950 50  0000 C CNN
 F 2 "~" H 4100 3100 60  0000 C CNN
@@
 	3250 1600 3250 1700
 Wire Wire Line
-	3050 1700 3250 1700
-Wire Wire Line
-	3250 1700 4250 1700
+	3050 1700 4250 1700
 Connection ~ 3250 1700
 Wire Wire Line
@@
 	4900 1700 4900 1150
 Wire Wire Line
-	3050 1900 3450 1900
-Wire Wire Line
-	3450 1900 4800 1900
+	3050 1900 4800 1900
 Wire Wire Line
 	3050 2100 5450 2100
@@
 	5500 1900 5500 1150
 $Comp
-L +12P #PWR?
+L +12P #PWR012
 U 1 1 523DFB91
 P 5500 1150
-F 0 "#PWR?" H 5500 1120 30  0001 C CNN
+F 0 "#PWR012" H 5500 1120 30  0001 C CNN
 F 1 "+12P" H 5500 1250 30  0000 C CNN
 F 2 "" H 5500 1150 60  0000 C CNN
@@
 $EndComp
 $Comp
-L -12P #PWR?
+L -12P #PWR013
 U 1 1 523E04D8
 P 6100 1150
-F 0 "#PWR?" H 6100 1280 20  0001 C CNN
+F 0 "#PWR013" H 6100 1280 20  0001 C CNN
 F 1 "-12P" H 6100 1250 30  0000 C CNN
 F 2 "" H 6100 1150 60  0000 C CNN
@@
 	6100 2100 5950 2100
 Wire Wire Line
-	2250 1600 2000 1600
-Wire Wire Line
-	2000 1600 1400 1600
+	1400 1600 2250 1600
 Wire Wire Line
 	2250 1700 2000 1700
@@
 	4800 3200 4800 3450
 $Comp
-L GND #PWR?
+L GND #PWR014
 U 1 1 523E08C4
 P 4800 3450
-F 0 "#PWR?" H 4800 3450 30  0001 C CNN
+F 0 "#PWR014" H 4800 3450 30  0001 C CNN
 F 1 "GND" H 4800 3380 30  0001 C CNN
 F 2 "" H 4800 3450 60  0000 C CNN
@@
 $EndComp
 $Comp
-L R R?
+L R R301
 U 1 1 523E08CC
 P 5150 3000
-F 0 "R?" V 5230 3000 40  0000 C CNN
+F 0 "R301" V 5230 3000 40  0000 C CNN
 F 1 "R" V 5157 3001 40  0000 C CNN
 F 2 "~" V 5080 3000 30  0000 C CNN
@@
 	5650 3000 5650 2750
 $Comp
-L +3.3V #PWR?
+L +3.3V #PWR015
 U 1 1 523E0910
 P 5650 2750
-F 0 "#PWR?" H 5650 2710 30  0001 C CNN
+F 0 "#PWR015" H 5650 2710 30  0001 C CNN
 F 1 "+3.3V" H 5650 2860 30  0000 C CNN
 F 2 "" H 5650 2750 60  0000 C CNN
@@
 $EndComp
 $Comp
-L +12P #PWR?
+L +12P #PWR016
 U 1 1 523E0C76
 P 8000 2250
-F 0 "#PWR?" H 8000 2220 30  0001 C CNN
+F 0 "#PWR016" H 8000 2220 30  0001 C CNN
 F 1 "+12P" H 8000 2350 30  0000 C CNN
 F 2 "" H 8000 2250 60  0000 C CNN
@@
 $EndComp
 $Comp
-L -12P #PWR?
+L -12P #PWR017
 U 1 1 523E0C7C
 P 8000 3800
-F 0 "#PWR?" H 8000 3930 20  0001 C CNN
+F 0 "#PWR017" H 8000 3930 20  0001 C CNN
 F 1 "-12P" H 8000 3900 30  0000 C CNN
 F 2 "" H 8000 3800 60  0000 C CNN
@@
 $EndComp
 $Comp
-L GND #PWR?
+L GND #PWR018
 U 1 1 523E0C82
 P 9000 3200
-F 0 "#PWR?" H 9000 3200 30  0001 C CNN
+F 0 "#PWR018" H 9000 3200 30  0001 C CNN
 F 1 "GND" H 9000 3130 30  0001 C CNN
 F 2 "" H 9000 3200 60  0000 C CNN
@@
 $EndComp
 $Comp
-L INDUCTOR L?
+L INDUCTOR L303
 U 1 1 523E0C8A
 P 8650 2450
-F 0 "L?" V 8600 2450 40  0000 C CNN
+F 0 "L303" V 8600 2450 40  0000 C CNN
 F 1 "INDUCTOR" V 8750 2450 40  0000 C CNN
 F 2 "~" H 8650 2450 60  0000 C CNN
@@
 $EndComp
 $Comp
-L INDUCTOR L?
+L INDUCTOR L302
 U 1 1 523E0C97
 P 8600 3650
-F 0 "L?" V 8550 3650 40  0000 C CNN
+F 0 "L302" V 8550 3650 40  0000 C CNN
 F 1 "INDUCTOR" V 8700 3650 40  0000 C CNN
 F 2 "~" H 8600 3650 60  0000 C CNN
@@
 $EndComp
 $Comp
-L C C?
+L C C302
 U 1 1 523E0C9F
 P 9450 2700
-F 0 "C?" H 9450 2800 40  0000 L CNN
+F 0 "C302" H 9450 2800 40  0000 L CNN
 F 1 "C" H 9456 2615 40  0000 L CNN
 F 2 "~" H 9488 2550 30  0000 C CNN
@@
 $EndComp
 $Comp
-L C C?
+L C C303
 U 1 1 523E0CAC
 P 9450 3350
-F 0 "C?" H 9450 3450 40  0000 L CNN
+F 0 "C303" H 9450 3450 40  0000 L CNN
 F 1 "C" H 9456 3265 40  0000 L CNN
 F 2 "~" H 9488 3200 30  0000 C CNN
@@
 	9450 3550 9450 3650
 Wire Wire Line
-	8900 3650 9450 3650
-Wire Wire Line
-	9450 3650 10350 3650
-Wire Wire Line
-	9450 2900 9450 3050
-Wire Wire Line
-	9450 3050 9450 3150
+	8900 3650 10350 3650
+Wire Wire Line
+	9450 2900 9450 3150
 Wire Wire Line
 	9450 2500 9450 2450
 Wire Wire Line
-	8950 2450 9450 2450
-Wire Wire Line
-	9450 2450 10350 2450
+	8950 2450 10350 2450
 Wire Wire Line
 	8000 2450 8350 2450
@@
 Connection ~ 9450 3050
 $Comp
-L -12V #PWR?
+L -12V #PWR019
 U 1 1 523E0DD3
 P 10350 3800
-F 0 "#PWR?" H 10350 3930 20  0001 C CNN
+F 0 "#PWR019" H 10350 3930 20  0001 C CNN
 F 1 "-12V" H 10350 3900 30  0000 C CNN
 F 2 "" H 10350 3800 60  0000 C CNN
@@
 Connection ~ 9450 2450
 $Comp
-L +12V #PWR?
+L +12V #PWR020
 U 1 1 523E0E37
 P 10350 2200
-F 0 "#PWR?" H 10350 2150 20  0001 C CNN
+F 0 "#PWR020" H 10350 2150 20  0001 C CNN
 F 1 "+12V" H 10350 2300 30  0000 C CNN
 F 2 "" H 10350 2200 60  0000 C CNN
@@
 Connection ~ 3450 1900
 $Comp
-L +12C #PWR?
+L +12C #PWR021
 U 1 1 52438F0D
 P 3450 1150
-F 0 "#PWR?" H 3450 1120 30  0001 C CNN
+F 0 "#PWR021" H 3450 1120 30  0001 C CNN
 F 1 "+12C" H 3450 1260 40  0000 C CNN
 F 2 "~" H 3450 1150 60  0000 C CNN
@@
 $EndComp
 $Comp
-L THERMISTOR TH?
+L THERMISTOR TH301
 U 1 1 52439695
 P 3900 1500
-F 0 "TH?" V 4000 1550 50  0000 C CNN
+F 0 "TH301" V 4000 1550 50  0000 C CNN
 F 1 "THERMISTOR" V 3800 1500 50  0000 C CNN
 F 2 "~" H 3900 1500 60  0000 C CNN
@@
 $EndComp
 $Comp
-L THERMISTOR TH?
+L THERMISTOR TH302
 U 1 1 524396A2
 P 4500 1700
-F 0 "TH?" V 4600 1750 50  0000 C CNN
+F 0 "TH302" V 4600 1750 50  0000 C CNN
 F 1 "THERMISTOR" V 4400 1700 50  0000 C CNN
 F 2 "~" H 4500 1700 60  0000 C CNN
@@
 $EndComp
 $Comp
-L THERMISTOR TH?
+L THERMISTOR TH303
 U 1 1 524396A8
 P 5050 1900
-F 0 "TH?" V 5150 1950 50  0000 C CNN
+F 0 "TH303" V 5150 1950 50  0000 C CNN
 F 1 "THERMISTOR" V 4950 1900 50  0000 C CNN
 F 2 "~" H 5050 1900 60  0000 C CNN
@@
 $EndComp
 $Comp
-L THERMISTOR TH?
+L THERMISTOR TH304
 U 1 1 524396AE
 P 5700 2100
-F 0 "TH?" V 5800 2150 50  0000 C CNN
+F 0 "TH304" V 5800 2150 50  0000 C CNN
 F 1 "THERMISTOR" V 5600 2100 50  0000 C CNN
 F 2 "~" H 5700 2100 60  0000 C CNN
@@
 $EndComp
 $Comp
-L GND #PWR?
+L GND #PWR022
 U 1 1 524502FC
 P 9400 1650
-F 0 "#PWR?" H 9400 1650 30  0001 C CNN
+F 0 "#PWR022" H 9400 1650 30  0001 C CNN
 F 1 "GND" H 9400 1580 30  0001 C CNN
 F 2 "" H 9400 1650 60  0000 C CNN
@@
 $EndComp
 $Comp
-L INDUCTOR L?
+L INDUCTOR L301
 U 1 1 52450302
 P 8600 900
-F 0 "L?" V 8550 900 40  0000 C CNN
+F 0 "L301" V 8550 900 40  0000 C CNN
 F 1 "INDUCTOR" V 8700 900 40  0000 C CNN
 F 2 "~" H 8600 900 60  0000 C CNN
@@
 $EndComp
 $Comp
-L C C?
+L C C301
 U 1 1 52450308
 P 9400 1150
-F 0 "C?" H 9400 1250 40  0000 L CNN
+F 0 "C301" H 9400 1250 40  0000 L CNN
 F 1 "C" H 9406 1065 40  0000 L CNN
 F 2 "~" H 9438 1000 30  0000 C CNN
@@
 	9400 950  9400 900
 Wire Wire Line
-	8900 900  9400 900
-Wire Wire Line
-	9400 900  10300 900
+	8900 900  10300 900
 Wire Wire Line
 	7950 900  8300 900
@@
 	7950 900  7950 700
 Wire Wire Line
-	9400 1650 9400 1500
-Wire Wire Line
-	9400 1500 9400 1500
+	9400 1350 9400 1650
 Connection ~ 9400 900
-Wire Wire Line
-	9400 1500 9400 1350
-$Comp
-L +5P #PWR?
+$Comp
+L +5P #PWR305
 U 1 1 52450355
 P 4900 1150
-F 0 "#PWR?" H 4900 1280 20  0001 C CNN
+F 0 "#PWR305" H 4900 1280 20  0001 C CNN
 F 1 "+5P" H 4900 1250 30  0000 C CNN
 F 2 "~" H 4900 1150 60  0000 C CNN
@@
 $EndComp
 $Comp
-L +3.3VP #PWR?
+L +3.3VP #PWR023
 U 1 1 52450364
 P 4400 1150
-F 0 "#PWR?" H 4450 1180 20  0001 C CNN
+F 0 "#PWR023" H 4450 1180 20  0001 C CNN
 F 1 "+3.3VP" H 4400 1240 30  0000 C CNN
 F 2 "~" H 4400 1150 60  0000 C CNN
@@
 $EndComp
 $Comp
-L +5P #PWR?
+L +5P #PWR309
 U 1 1 52450371
 P 7950 700
-F 0 "#PWR?" H 7950 830 20  0001 C CNN
+F 0 "#PWR309" H 7950 830 20  0001 C CNN
 F 1 "+5P" H 7950 800 30  0000 C CNN
 F 2 "~" H 7950 700 60  0000 C CNN
@@
 $EndComp
 $Comp
-L +5V #PWR?
+L +5V #PWR024
 U 1 1 524503B6
 P 10300 650
-F 0 "#PWR?" H 10300 740 20  0001 C CNN
+F 0 "#PWR024" H 10300 740 20  0001 C CNN
 F 1 "+5V" H 10300 740 30  0000 C CNN
 F 2 "~" H 10300 650 60  0000 C CNN

Commit message: syncing to upstream
Parts:
- renumbered C301 to C2, C302 to C3, C303 to C4, L301 to L1, L302 to L2, L303 to L3, P301 to P1, R301 to R14, SW301 to SW1, TH301 to TH1, TH302 to TH2, TH303 to TH3, TH304 to TH4
Changed lines of the file:
@@
-EESchema Schematic File Version 2
+EESchema Schematic File Version 2  date 10/10/2013 1:06:29 AM
 LIBS:power
 LIBS:device
@@
 Sheet 3 9
 Title ""
-Date "3 mar 2014"
+Date "10 oct 2013"
 Rev ""
 Comp ""
@@
 $EndDescr
 $Comp
-L CONN_12X2 P301
+L CONN_12X2 P1
 U 1 1 523DFA5D
 P 2650 2050
-F 0 "P301" H 2650 2700 60  0000 C CNN
+F 0 "P1" H 2650 2700 60  0000 C CNN
 F 1 "CONN_12X2" V 2650 2050 50  0000 C CNN
 F 2 "" H 2650 2050 60  0000 C CNN
@@
 $EndComp
 $Comp
-L GND #PWR011
+L GND #PWR11
 U 1 1 523DFA76
 P 1400 1850
-F 0 "#PWR011" H 1400 1850 30  0001 C CNN
+F 0 "#PWR11" H 1400 1850 30  0001 C CNN
 F 1 "GND" H 1400 1780 30  0001 C CNN
 F 2 "" H 1400 1850 60  0000 C CNN
@@
 $EndComp
 $Comp
-L SWITCH_INV SW301
+L SWITCH_INV SW1
 U 1 1 523DFB25
 P 4100 3100
-F 0 "SW301" H 3900 3250 50  0000 C CNN
+F 0 "SW1" H 3900 3250 50  0000 C CNN
 F 1 "SWITCH_INV" H 3950 2950 50  0000 C CNN
 F 2 "~" H 4100 3100 60  0000 C CNN
@@
 	5500 1900 5500 1150
 $Comp
-L +12P #PWR012
+L +12P #PWR16
 U 1 1 523DFB91
 P 5500 1150
-F 0 "#PWR012" H 5500 1120 30  0001 C CNN
+F 0 "#PWR16" H 5500 1120 30  0001 C CNN
 F 1 "+12P" H 5500 1250 30  0000 C CNN
 F 2 "" H 5500 1150 60  0000 C CNN
@@
 $EndComp
 $Comp
-L -12P #PWR013
+L -12P #PWR18
 U 1 1 523E04D8
 P 6100 1150
-F 0 "#PWR013" H 6100 1280 20  0001 C CNN
+F 0 "#PWR18" H 6100 1280 20  0001 C CNN
 F 1 "-12P" H 6100 1250 30  0000 C CNN
 F 2 "" H 6100 1150 60  0000 C CNN
@@
 	4800 3200 4800 3450
 $Comp
-L GND #PWR014
+L GND #PWR14
 U 1 1 523E08C4
 P 4800 3450
-F 0 "#PWR014" H 4800 3450 30  0001 C CNN
+F 0 "#PWR14" H 4800 3450 30  0001 C CNN
 F 1 "GND" H 4800 3380 30  0001 C CNN
 F 2 "" H 4800 3450 60  0000 C CNN
@@
 $EndComp
 $Comp
-L R R301
+L R R14
 U 1 1 523E08CC
 P 5150 3000
-F 0 "R301" V 5230 3000 40  0000 C CNN
+F 0 "R14" V 5230 3000 40  0000 C CNN
 F 1 "R" V 5157 3001 40  0000 C CNN
 F 2 "~" V 5080 3000 30  0000 C CNN
@@
 	5650 3000 5650 2750
 $Comp
-L +3.3V #PWR015
+L +3.3V #PWR17
 U 1 1 523E0910
 P 5650 2750
-F 0 "#PWR015" H 5650 2710 30  0001 C CNN
+F 0 "#PWR17" H 5650 2710 30  0001 C CNN
 F 1 "+3.3V" H 5650 2860 30  0000 C CNN
 F 2 "" H 5650 2750 60  0000 C CNN
@@
 $EndComp
 $Comp
-L +12P #PWR016
+L +12P #PWR20
 U 1 1 523E0C76
 P 8000 2250
-F 0 "#PWR016" H 8000 2220 30  0001 C CNN
+F 0 "#PWR20" H 8000 2220 30  0001 C CNN
 F 1 "+12P" H 8000 2350 30  0000 C CNN
 F 2 "" H 8000 2250 60  0000 C CNN
@@
 $EndComp
 $Comp
-L -12P #PWR017
+L -12P #PWR21
 U 1 1 523E0C7C
 P 8000 3800
-F 0 "#PWR017" H 8000 3930 20  0001 C CNN
+F 0 "#PWR21" H 8000 3930 20  0001 C CNN
 F 1 "-12P" H 8000 3900 30  0000 C CNN
 F 2 "" H 8000 3800 60  0000 C CNN
@@
 $EndComp
 $Comp
-L GND #PWR018
+L GND #PWR22
 U 1 1 523E0C82
 P 9000 3200
-F 0 "#PWR018" H 9000 3200 30  0001 C CNN
+F 0 "#PWR22" H 9000 3200 30  0001 C CNN
 F 1 "GND" H 9000 3130 30  0001 C CNN
 F 2 "" H 9000 3200 60  0000 C CNN
@@
 $EndComp
 $Comp
-L INDUCTOR L303
+L INDUCTOR L3
 U 1 1 523E0C8A
 P 8650 2450
-F 0 "L303" V 8600 2450 40  0000 C CNN
+F 0 "L3" V 8600 2450 40  0000 C CNN
 F 1 "INDUCTOR" V 8750 2450 40  0000 C CNN
 F 2 "~" H 8650 2450 60  0000 C CNN
@@
 $EndComp
 $Comp
-L INDUCTOR L302
+L INDUCTOR L2
 U 1 1 523E0C97
 P 8600 3650
-F 0 "L302" V 8550 3650 40  0000 C CNN
+F 0 "L2" V 8550 3650 40  0000 C CNN
 F 1 "INDUCTOR" V 8700 3650 40  0000 C CNN
 F 2 "~" H 8600 3650 60  0000 C CNN
@@
 $EndComp
 $Comp
-L C C302
+L C C3
 U 1 1 523E0C9F
 P 9450 2700
-F 0 "C302" H 9450 2800 40  0000 L CNN
+F 0 "C3" H 9450 2800 40  0000 L CNN
 F 1 "C" H 9456 2615 40  0000 L CNN
 F 2 "~" H 9488 2550 30  0000 C CNN
@@
 $EndComp
 $Comp
-L C C303
+L C C4
 U 1 1 523E0CAC
 P 9450 3350
-F 0 "C303" H 9450 3450 40  0000 L CNN
+F 0 "C4" H 9450 3450 40  0000 L CNN
 F 1 "C" H 9456 3265 40  0000 L CNN
 F 2 "~" H 9488 3200 30  0000 C CNN
@@
 Connection ~ 9450 3050
 $Comp
-L -12V #PWR019
+L -12V #PWR26
 U 1 1 523E0DD3
 P 10350 3800
-F 0 "#PWR019" H 10350 3930 20  0001 C CNN
+F 0 "#PWR26" H 10350 3930 20  0001 C CNN
 F 1 "-12V" H 10350 3900 30  0000 C CNN
 F 2 "" H 10350 3800 60  0000 C CNN
@@
 Connection ~ 9450 2450
 $Comp
-L +12V #PWR020
+L +12V #PWR25
 U 1 1 523E0E37
 P 10350 2200
-F 0 "#PWR020" H 10350 2150 20  0001 C CNN
+F 0 "#PWR25" H 10350 2150 20  0001 C CNN
 F 1 "+12V" H 10350 2300 30  0000 C CNN
 F 2 "" H 10350 2200 60  0000 C CNN
@@
 Connection ~ 3450 1900
 $Comp
-L +12C #PWR021
+L +12C #PWR12
 U 1 1 52438F0D
 P 3450 1150
-F 0 "#PWR021" H 3450 1120 30  0001 C CNN
+F 0 "#PWR12" H 3450 1120 30  0001 C CNN
 F 1 "+12C" H 3450 1260 40  0000 C CNN
 F 2 "~" H 3450 1150 60  0000 C CNN
@@
 $EndComp
 $Comp
-L THERMISTOR TH301
+L THERMISTOR TH1
 U 1 1 52439695
 P 3900 1500
-F 0 "TH301" V 4000 1550 50  0000 C CNN
+F 0 "TH1" V 4000 1550 50  0000 C CNN
 F 1 "THERMISTOR" V 3800 1500 50  0000 C CNN
 F 2 "~" H 3900 1500 60  0000 C CNN
@@
 $EndComp
 $Comp
-L THERMISTOR TH302
+L THERMISTOR TH2
 U 1 1 524396A2
 P 4500 1700
-F 0 "TH302" V 4600 1750 50  0000 C CNN
+F 0 "TH2" V 4600 1750 50  0000 C CNN
 F 1 "THERMISTOR" V 4400 1700 50  0000 C CNN
 F 2 "~" H 4500 1700 60  0000 C CNN
@@
 $EndComp
 $Comp
-L THERMISTOR TH303
+L THERMISTOR TH3
 U 1 1 524396A8
 P 5050 1900
-F 0 "TH303" V 5150 1950 50  0000 C CNN
+F 0 "TH3" V 5150 1950 50  0000 C CNN
 F 1 "THERMISTOR" V 4950 1900 50  0000 C CNN
 F 2 "~" H 5050 1900 60  0000 C CNN
@@
 $EndComp
 $Comp
-L THERMISTOR TH304
+L THERMISTOR TH4
 U 1 1 524396AE
 P 5700 2100
-F 0 "TH304" V 5800 2150 50  0000 C CNN
+F 0 "TH4" V 5800 2150 50  0000 C CNN
 F 1 "THERMISTOR" V 5600 2100 50  0000 C CNN
 F 2 "~" H 5700 2100 60  0000 C CNN
@@
 $EndComp
 $Comp
-L GND #PWR022
+L GND #PWR23
 U 1 1 524502FC
 P 9400 1650
-F 0 "#PWR022" H 9400 1650 30  0001 C CNN
+F 0 "#PWR23" H 9400 1650 30  0001 C CNN
 F 1 "GND" H 9400 1580 30  0001 C CNN
 F 2 "" H 9400 1650 60  0000 C CNN
@@
 $EndComp
 $Comp
-L INDUCTOR L301
+L INDUCTOR L1
 U 1 1 52450302
 P 8600 900
-F 0 "L301" V 8550 900 40  0000 C CNN
+F 0 "L1" V 8550 900 40  0000 C CNN
 F 1 "INDUCTOR" V 8700 900 40  0000 C CNN
 F 2 "~" H 8600 900 60  0000 C CNN
@@
 $EndComp
 $Comp
-L C C301
+L C C2
 U 1 1 52450308
 P 9400 1150
-F 0 "C301" H 9400 1250 40  0000 L CNN
+F 0 "C2" H 9400 1250 40  0000 L CNN
 F 1 "C" H 9406 1065 40  0000 L CNN
 F 2 "~" H 9438 1000 30  0000 C CNN
@@
 Connection ~ 9400 900
 $Comp
-L +5P #PWR305
+L +5P #PWR15
 U 1 1 52450355
 P 4900 1150
-F 0 "#PWR305" H 4900 1280 20  0001 C CNN
+F 0 "#PWR15" H 4900 1280 20  0001 C CNN
 F 1 "+5P" H 4900 1250 30  0000 C CNN
 F 2 "~" H 4900 1150 60  0000 C CNN
@@
 $EndComp
 $Comp
-L +3.3VP #PWR023
+L +3.3VP #PWR13
 U 1 1 52450364
 P 4400 1150
-F 0 "#PWR023" H 4450 1180 20  0001 C CNN
+F 0 "#PWR13" H 4450 1180 20  0001 C CNN
 F 1 "+3.3VP" H 4400 1240 30  0000 C CNN
 F 2 "~" H 4400 1150 60  0000 C CNN
@@
 $EndComp
 $Comp
-L +5P #PWR309
+L +5P #PWR19
 U 1 1 52450371
 P 7950 700
-F 0 "#PWR309" H 7950 830 20  0001 C CNN
+F 0 "#PWR19" H 7950 830 20  0001 C CNN
 F 1 "+5P" H 7950 800 30  0000 C CNN
 F 2 "~" H 7950 700 60  0000 C CNN
@@
 $EndComp
 $Comp
-L +5V #PWR024
+L +5V #PWR24
 U 1 1 524503B6
 P 10300 650
-F 0 "#PWR024" H 10300 740 20  0001 C CNN
+F 0 "#PWR24" H 10300 740 20  0001 C CNN
 F 1 "+5V" H 10300 740 30  0000 C CNN
 F 2 "~" H 10300 650 60  0000 C CNN
