File: BenchBudEE/PowerAdjustmentMonitor.sch (KiCad schematic (older format))
At the start: 29 parts

Commit message: checking in all my local changes before syncing to chris's repo.
Parts:
- gave numbers to parts that had none: 28
Connections:
- net V+_CURR_MON: now also U7.6 (-), U7.7; no longer U7.1, U7.2 (-)
- net V-_CURR_MON: now also U7.8, U7.9 (-); no longer U7.1, U7.2 (-)
