File: BenchBudEE/PowerAdjustmentMonitor.sch (KiCad schematic (older format))
At the start: 8 parts

Commit message: swapping Power and PowerAdjustmentMonitor schematics
Parts:
- removed C?: 5566-20A, ~, symbol 5566-20A
- removed F? (x6): FUSE, ~, symbol FUSE
- removed SW?: SWITCH_INV, ~, symbol SWITCH_INV
Connections:
- net labels removed: +12V, +3.3V, +5V, -12V, -5V, GND
- wire segments 35 -> 0

Commit message: Implementing current control and monitor schematic.
Parts:
- added C? (x8): CP1, ~, symbol CP1
- added JP?: JUMPER, ~, symbol JUMPER
- added R? (x10): R, ~, symbol R
- added RV? (x2): POT, ~, symbol POT
- added U? (x2): LM317, ~, symbol LM317
- added U? (x2): LM337T, TO-220, symbol LM337T
Connections:
- net labels added: -12V_FILTERED, -12V_REGULATED, 12V_FILTERED, 12V_REGULATED, 3.3V_FUSED, 3V3_MON, 5V_FUSED, 5V_MON, AGND, GND, V+_ADJ, V+_ADJ_MON, V-_ADJ, V-_ADJ_MON
- wire segments 0 -> 90

Commit message: Completing schematics from week 3 videos.
Parts:
- added R? (x2): R, ~, symbol R
- added U? (x2): LM324, symbol LM324
Connections:
- net labels added: 12v_FILTERED, V+_CURR_MON, V-_CURR_MON
- wire segments 90 -> 114
Other:
- moved on the sheet: R?

Commit message: syncing to https://github.com/ContextualElectronics/BenchBudEE/tree/ebd662c68b928f78643cdf924dc35a4d91f03121
Parts:
- removed C? (x8): CP1, ~, symbol CP1
- removed JP?: JUMPER, ~, symbol JUMPER
- removed R? (x12): R, ~, symbol R
- removed RV? (x2): POT, ~, symbol POT
- removed U? (x2): LM317, ~, symbol LM317
- removed U? (x2): LM337T, TO-220, symbol LM337T
- removed U? (x2): LM324, symbol LM324
- added JP? (x3): JUMPER, ~, symbol JUMPER
- added R? (x6): R, ~, symbol R
- added R? (x2): RVAR, ~, symbol RVAR
- added U? (x2): LM317, ~, symbol LM317
- added U? (x2): 7805, ~, symbol 7805
Connections:
- net labels added: +12V, +3.3V, +5V, -12V, FE_V+, FE_V-, V+_MON, V-_MON
- net labels removed: -12V_FILTERED, -12V_REGULATED, 12V_FILTERED, 12V_REGULATED, 12v_FILTERED, 3.3V_FUSED, 5V_FUSED, V+_CURR_MON, V-_CURR_MON
- wire segments 114 -> 57

Commit message: playing with the layout
Parts:
- gave numbers to parts that had none: 15
Changed lines of the file:
@@
-EESchema Schematic File Version 2  date 10/10/2013 12:18:22 AM
+EESchema Schematic File Version 2
 LIBS:power
 LIBS:device
@@
 Sheet 7 9
 Title ""
-Date "10 oct 2013"
+Date "3 mar 2014"
 Rev ""
 Comp ""
@@
 $EndDescr
 $Comp
-L +3.3V #PWR?
+L +3.3V #PWR036
 U 1 1 523E00C5
 P 9000 2250
-F 0 "#PWR?" H 9000 2210 30  0001 C CNN
+F 0 "#PWR036" H 9000 2210 30  0001 C CNN
 F 1 "+3.3V" H 9000 2360 30  0000 C CNN
 F 2 "" H 9000 2250 60  0000 C CNN
@@
 $EndComp
 $Comp
-L +5V #PWR?
+L +5V #PWR037
 U 1 1 523E00CB
 P 8700 2250
-F 0 "#PWR?" H 8700 2340 20  0001 C CNN
+F 0 "#PWR037" H 8700 2340 20  0001 C CNN
 F 1 "+5V" H 8700 2340 30  0000 C CNN
 F 2 "" H 8700 2250 60  0000 C CNN
@@
 $EndComp
 $Comp
-L -12V #PWR?
+L -12V #PWR038
 U 1 1 523E0153
 P 2200 5250
-F 0 "#PWR?" H 2200 5380 20  0001 C CNN
+F 0 "#PWR038" H 2200 5380 20  0001 C CNN
 F 1 "-12V" H 2200 5350 30  0000 C CNN
 F 2 "" H 2200 5250 60  0000 C CNN
@@
 $EndComp
 $Comp
-L +12V #PWR?
+L +12V #PWR039
 U 1 1 523E015D
 P 2200 3300
-F 0 "#PWR?" H 2200 3250 20  0001 C CNN
+F 0 "#PWR039" H 2200 3250 20  0001 C CNN
 F 1 "+12V" H 2200 3400 30  0000 C CNN
 F 2 "" H 2200 3300 60  0000 C CNN
@@
 $EndComp
 $Comp
-L LM317 U?
+L LM317 U703
 U 1 1 523E0682
 P 3300 7100
-F 0 "U?" H 3300 7400 60  0000 C CNN
+F 0 "U703" H 3300 7400 60  0000 C CNN
 F 1 "LM317" H 3350 6850 60  0000 L CNN
 F 2 "~" H 3300 7100 60  0000 C CNN
@@
 $EndComp
 $Comp
-L JUMPER JP?
+L JUMPER JP702
 U 1 1 523E069B
 P 3300 2950
-F 0 "JP?" H 3300 3100 60  0000 C CNN
+F 0 "JP702" H 3300 3100 60  0000 C CNN
 F 1 "JUMPER" H 3300 2870 40  0000 C CNN
 F 2 "~" H 3300 2950 60  0000 C CNN
@@
 $EndComp
 $Comp
-L JUMPER JP?
+L JUMPER JP703
 U 1 1 523E06A8
 P 3300 5450
-F 0 "JP?" H 3300 5600 60  0000 C CNN
+F 0 "JP703" H 3300 5600 60  0000 C CNN
 F 1 "JUMPER" H 3300 5370 40  0000 C CNN
 F 2 "~" H 3300 5450 60  0000 C CNN
@@
 $EndComp
 $Comp
-L GND #PWR?
+L GND #PWR040
 U 1 1 523E06F9
 P 1100 4600
-F 0 "#PWR?" H 1100 4600 30  0001 C CNN
+F 0 "#PWR040" H 1100 4600 30  0001 C CNN
 F 1 "GND" H 1100 4530 30  0001 C CNN
 F 2 "~" H 1100 4600 60  0000 C CNN
@@
 $EndComp
 $Comp
-L AGND #PWR?
+L AGND #PWR041
 U 1 1 523E08B2
 P 1700 4600
-F 0 "#PWR?" H 1700 4600 40  0001 C CNN
+F 0 "#PWR041" H 1700 4600 40  0001 C CNN
 F 1 "AGND" H 1700 4530 50  0000 C CNN
 F 2 "~" H 1700 4600 60  0000 C CNN
@@
 $EndComp
 $Comp
-L JUMPER JP?
+L JUMPER JP701
 U 1 1 523E08BF
 P 1400 4250
-F 0 "JP?" H 1400 4400 60  0000 C CNN
+F 0 "JP701" H 1400 4400 60  0000 C CNN
 F 1 "JUMPER" H 1400 4170 40  0000 C CNN
 F 2 "~" H 1400 4250 60  0000 C CNN
@@
 $EndComp
 $Comp
-L AGND #PWR?
+L AGND #PWR042
 U 1 1 52562CAD
 P 2500 4400
-F 0 "#PWR?" H 2500 4400 40  0001 C CNN
+F 0 "#PWR042" H 2500 4400 40  0001 C CNN
 F 1 "AGND" H 2500 4330 50  0000 C CNN
 F 2 "~" H 2500 4400 60  0000 C CNN
@@
 $EndComp
 $Comp
-L FE_V+ #PWR?
+L FE_V+ #PWR043
 U 1 1 523E0975
 P 4200 2800
-F 0 "#PWR?" H 4200 2900 30  0001 C CNN
+F 0 "#PWR043" H 4200 2900 30  0001 C CNN
 F 1 "FE_V+" H 4200 2900 30  0000 C CNN
 F 2 "~" H 4200 2800 60  0000 C CNN
@@
 $EndComp
 $Comp
-L FE_V- #PWR?
+L FE_V- #PWR709
 U 1 1 523E099B
 P 4250 5600
-F 0 "#PWR?" H 4250 5800 40  0001 C CNN
+F 0 "#PWR709" H 4250 5800 40  0001 C CNN
 F 1 "FE_V-" H 4250 5750 40  0000 C CNN
 F 2 "~" H 4250 5600 60  0000 C CNN
@@
 $EndComp
 $Comp
-L 7805 U?
+L 7805 U701
 U 1 1 523E09EA
 P 3300 3500
-F 0 "U?" H 3450 3304 60  0000 C CNN
+F 0 "U701" H 3450 3304 60  0000 C CNN
 F 1 "7805" H 3300 3700 60  0000 C CNN
 F 2 "~" H 3300 3500 60  0000 C CNN
@@
 $EndComp
 $Comp
-L 7805 U?
+L 7805 U702
 U 1 1 523E09F7
 P 3300 4950
-F 0 "U?" H 3450 4754 60  0000 C CNN
+F 0 "U702" H 3450 4754 60  0000 C CNN
 F 1 "7805" H 3300 5150 60  0000 C CNN
 F 2 "~" H 3300 4950 60  0000 C CNN
@@
 $EndComp
 $Comp
-L R R?
+L R R701
 U 1 1 523E0AC1
 P 3900 6350
-F 0 "R?" V 3980 6350 40  0000 C CNN
+F 0 "R701" V 3980 6350 40  0000 C CNN
 F 1 "R" V 3907 6351 40  0000 C CNN
 F 2 "~" V 3830 6350 30  0000 C CNN
@@
 $EndComp
 $Comp
-L AGND #PWR?
+L AGND #PWR044
 U 1 1 523E0B09
 P 3600 6100
-F 0 "#PWR?" H 3600 6100 40  0001 C CNN
+F 0 "#PWR044" H 3600 6100 40  0001 C CNN
 F 1 "AGND" H 3600 6030 50  0000 C CNN
 F 2 "~" H 3600 6100 60  0000 C CNN
@@
 $EndComp
 $Comp
-L LM317 U?
+L LM317 U704
 U 1 1 523E0B74
 P 3350 1100
-F 0 "U?" H 3350 1400 60  0000 C CNN
+F 0 "U704" H 3350 1400 60  0000 C CNN
 F 1 "LM317" H 3400 850 60  0000 L CNN
 F 2 "~" H 3350 1100 60  0000 C CNN
@@
 $EndComp
 $Comp
-L R R?
+L R R704
 U 1 1 523E0B81
 P 3950 1850
-F 0 "R?" V 4030 1850 40  0000 C CNN
+F 0 "R704" V 4030 1850 40  0000 C CNN
 F 1 "R" V 3957 1851 40  0000 C CNN
 F 2 "~" V 3880 1850 30  0000 C CNN
@@
 $EndComp
 $Comp
-L AGND #PWR?
+L AGND #PWR045
 U 1 1 523E0B8A
 P 3950 2250
-F 0 "#PWR?" H 3950 2250 40  0001 C CNN
+F 0 "#PWR045" H 3950 2250 40  0001 C CNN
 F 1 "AGND" H 3950 2180 50  0000 C CNN
 F 2 "~" H 3950 2250 60  0000 C CNN
@@
 V-_ADJ_MON
 $Comp
-L R R?
+L R R705
 U 1 1 523E1074
 P 6500 2750
-F 0 "R?" V 6580 2750 40  0000 C CNN
+F 0 "R705" V 6580 2750 40  0000 C CNN
 F 1 "R" V 6507 2751 40  0000 C CNN
 F 2 "~" V 6430 2750 30  0000 C CNN
@@
 $EndComp
 $Comp
-L R R?
+L R R706
 U 1 1 523E107A
 P 6500 3400
-F 0 "R?" V 6580 3400 40  0000 C CNN
+F 0 "R706" V 6580 3400 40  0000 C CNN
 F 1 "R" V 6507 3401 40  0000 C CNN
 F 2 "~" V 6430 3400 30  0000 C CNN
@@
 $EndComp
 $Comp
-L R R?
+L R R707
 U 1 1 523E114C
 P 6500 4700
-F 0 "R?" V 6580 4700 40  0000 C CNN
+F 0 "R707" V 6580 4700 40  0000 C CNN
 F 1 "R" V 6507 4701 40  0000 C CNN
 F 2 "~" V 6430 4700 30  0000 C CNN
@@
 $EndComp
 $Comp
-L R R?
+L R R708
 U 1 1 523E1152
 P 6500 5400
-F 0 "R?" V 6580 5400 40  0000 C CNN
+F 0 "R708" V 6580 5400 40  0000 C CNN
 F 1 "R" V 6507 5401 40  0000 C CNN
 F 2 "~" V 6430 5400 30  0000 C CNN
@@
 	6500 3050 9350 3050
 $Comp
-L RVAR R?
+L RVAR R702
 U 1 1 523E21E8
 P 3900 6950
-F 0 "R?" V 3980 6900 50  0000 C CNN
+F 0 "R702" V 3980 6900 50  0000 C CNN
 F 1 "RVAR" V 3820 7010 50  0000 C CNN
 F 2 "~" H 3900 6950 60  0000 C CNN
@@
 $EndComp
 $Comp
-L RVAR R?
+L RVAR R703
 U 1 1 523E21FB
 P 3950 1250
-F 0 "R?" V 4030 1200 50  0000 C CNN
+F 0 "R703" V 4030 1200 50  0000 C CNN
 F 1 "RVAR" V 3870 1310 50  0000 C CNN
 F 2 "~" H 3950 1250 60  0000 C CNN

Commit message: syncing to upstream
Parts:
- renumbered JP701 to JP1, JP702 to JP2, JP703 to JP3, R701 to R18, R702 to R19, R703 to R20, R704 to R21, R705 to R22, R706 to R23, R707 to R24, R708 to R25, U703 to U10, U704 to U11, U701 to U8, U702 to U9
Changed lines of the file:
@@
-EESchema Schematic File Version 2
+EESchema Schematic File Version 2  date 10/10/2013 1:06:29 AM
 LIBS:power
 LIBS:device
@@
 Sheet 7 9
 Title ""
-Date "3 mar 2014"
+Date "10 oct 2013"
 Rev ""
 Comp ""
@@
 $EndDescr
 $Comp
-L +3.3V #PWR036
+L +3.3V #PWR48
 U 1 1 523E00C5
 P 9000 2250
-F 0 "#PWR036" H 9000 2210 30  0001 C CNN
+F 0 "#PWR48" H 9000 2210 30  0001 C CNN
 F 1 "+3.3V" H 9000 2360 30  0000 C CNN
 F 2 "" H 9000 2250 60  0000 C CNN
@@
 $EndComp
 $Comp
-L +5V #PWR037
+L +5V #PWR47
 U 1 1 523E00CB
 P 8700 2250
-F 0 "#PWR037" H 8700 2340 20  0001 C CNN
+F 0 "#PWR47" H 8700 2340 20  0001 C CNN
 F 1 "+5V" H 8700 2340 30  0000 C CNN
 F 2 "" H 8700 2250 60  0000 C CNN
@@
 $EndComp
 $Comp
-L -12V #PWR038
+L -12V #PWR41
 U 1 1 523E0153
 P 2200 5250
-F 0 "#PWR038" H 2200 5380 20  0001 C CNN
+F 0 "#PWR41" H 2200 5380 20  0001 C CNN
 F 1 "-12V" H 2200 5350 30  0000 C CNN
 F 2 "" H 2200 5250 60  0000 C CNN
@@
 $EndComp
 $Comp
-L +12V #PWR039
+L +12V #PWR40
 U 1 1 523E015D
 P 2200 3300
-F 0 "#PWR039" H 2200 3250 20  0001 C CNN
+F 0 "#PWR40" H 2200 3250 20  0001 C CNN
 F 1 "+12V" H 2200 3400 30  0000 C CNN
 F 2 "" H 2200 3300 60  0000 C CNN
@@
 $EndComp
 $Comp
-L LM317 U703
+L LM317 U10
 U 1 1 523E0682
 P 3300 7100
-F 0 "U703" H 3300 7400 60  0000 C CNN
+F 0 "U10" H 3300 7400 60  0000 C CNN
 F 1 "LM317" H 3350 6850 60  0000 L CNN
 F 2 "~" H 3300 7100 60  0000 C CNN
@@
 $EndComp
 $Comp
-L JUMPER JP702
+L JUMPER JP2
 U 1 1 523E069B
 P 3300 2950
-F 0 "JP702" H 3300 3100 60  0000 C CNN
+F 0 "JP2" H 3300 3100 60  0000 C CNN
 F 1 "JUMPER" H 3300 2870 40  0000 C CNN
 F 2 "~" H 3300 2950 60  0000 C CNN
@@
 $EndComp
 $Comp
-L JUMPER JP703
+L JUMPER JP3
 U 1 1 523E06A8
 P 3300 5450
-F 0 "JP703" H 3300 5600 60  0000 C CNN
+F 0 "JP3" H 3300 5600 60  0000 C CNN
 F 1 "JUMPER" H 3300 5370 40  0000 C CNN
 F 2 "~" H 3300 5450 60  0000 C CNN
@@
 $EndComp
 $Comp
-L GND #PWR040
+L GND #PWR38
 U 1 1 523E06F9
 P 1100 4600
-F 0 "#PWR040" H 1100 4600 30  0001 C CNN
+F 0 "#PWR38" H 1100 4600 30  0001 C CNN
 F 1 "GND" H 1100 4530 30  0001 C CNN
 F 2 "~" H 1100 4600 60  0000 C CNN
@@
 $EndComp
 $Comp
-L AGND #PWR041
+L AGND #PWR39
 U 1 1 523E08B2
 P 1700 4600
-F 0 "#PWR041" H 1700 4600 40  0001 C CNN
+F 0 "#PWR39" H 1700 4600 40  0001 C CNN
 F 1 "AGND" H 1700 4530 50  0000 C CNN
 F 2 "~" H 1700 4600 60  0000 C CNN
@@
 $EndComp
 $Comp
-L JUMPER JP701
+L JUMPER JP1
 U 1 1 523E08BF
 P 1400 4250
-F 0 "JP701" H 1400 4400 60  0000 C CNN
+F 0 "JP1" H 1400 4400 60  0000 C CNN
 F 1 "JUMPER" H 1400 4170 40  0000 C CNN
 F 2 "~" H 1400 4250 60  0000 C CNN
@@
 $EndComp
 $Comp
-L AGND #PWR042
+L AGND #PWR42
 U 1 1 52562CAD
 P 2500 4400
-F 0 "#PWR042" H 2500 4400 40  0001 C CNN
+F 0 "#PWR42" H 2500 4400 40  0001 C CNN
 F 1 "AGND" H 2500 4330 50  0000 C CNN
 F 2 "~" H 2500 4400 60  0000 C CNN
@@
 $EndComp
 $Comp
-L FE_V+ #PWR043
+L FE_V+ #PWR45
 U 1 1 523E0975
 P 4200 2800
-F 0 "#PWR043" H 4200 2900 30  0001 C CNN
+F 0 "#PWR45" H 4200 2900 30  0001 C CNN
 F 1 "FE_V+" H 4200 2900 30  0000 C CNN
 F 2 "~" H 4200 2800 60  0000 C CNN
@@
 $EndComp
 $Comp
-L FE_V- #PWR709
+L FE_V- #PWR46
 U 1 1 523E099B
 P 4250 5600
-F 0 "#PWR709" H 4250 5800 40  0001 C CNN
+F 0 "#PWR46" H 4250 5800 40  0001 C CNN
 F 1 "FE_V-" H 4250 5750 40  0000 C CNN
 F 2 "~" H 4250 5600 60  0000 C CNN
@@
 $EndComp
 $Comp
-L 7805 U701
+L 7805 U8
 U 1 1 523E09EA
 P 3300 3500
-F 0 "U701" H 3450 3304 60  0000 C CNN
+F 0 "U8" H 3450 3304 60  0000 C CNN
 F 1 "7805" H 3300 3700 60  0000 C CNN
 F 2 "~" H 3300 3500 60  0000 C CNN
@@
 $EndComp
 $Comp
-L 7805 U702
+L 7805 U9
 U 1 1 523E09F7
 P 3300 4950
-F 0 "U702" H 3450 4754 60  0000 C CNN
+F 0 "U9" H 3450 4754 60  0000 C CNN
 F 1 "7805" H 3300 5150 60  0000 C CNN
 F 2 "~" H 3300 4950 60  0000 C CNN
@@
 $EndComp
 $Comp
-L R R701
+L R R18
 U 1 1 523E0AC1
 P 3900 6350
-F 0 "R701" V 3980 6350 40  0000 C CNN
+F 0 "R18" V 3980 6350 40  0000 C CNN
 F 1 "R" V 3907 6351 40  0000 C CNN
 F 2 "~" V 3830 6350 30  0000 C CNN
@@
 $EndComp
 $Comp
-L AGND #PWR044
+L AGND #PWR43
 U 1 1 523E0B09
 P 3600 6100
-F 0 "#PWR044" H 3600 6100 40  0001 C CNN
+F 0 "#PWR43" H 3600 6100 40  0001 C CNN
 F 1 "AGND" H 3600 6030 50  0000 C CNN
 F 2 "~" H 3600 6100 60  0000 C CNN
@@
 $EndComp
 $Comp
-L LM317 U704
+L LM317 U11
 U 1 1 523E0B74
 P 3350 1100
-F 0 "U704" H 3350 1400 60  0000 C CNN
+F 0 "U11" H 3350 1400 60  0000 C CNN
 F 1 "LM317" H 3400 850 60  0000 L CNN
 F 2 "~" H 3350 1100 60  0000 C CNN
@@
 $EndComp
 $Comp
-L R R704
+L R R21
 U 1 1 523E0B81
 P 3950 1850
-F 0 "R704" V 4030 1850 40  0000 C CNN
+F 0 "R21" V 4030 1850 40  0000 C CNN
 F 1 "R" V 3957 1851 40  0000 C CNN
 F 2 "~" V 3880 1850 30  0000 C CNN
@@
 $EndComp
 $Comp
-L AGND #PWR045
+L AGND #PWR44
 U 1 1 523E0B8A
 P 3950 2250
-F 0 "#PWR045" H 3950 2250 40  0001 C CNN
+F 0 "#PWR44" H 3950 2250 40  0001 C CNN
 F 1 "AGND" H 3950 2180 50  0000 C CNN
 F 2 "~" H 3950 2250 60  0000 C CNN
@@
 V-_ADJ_MON
 $Comp
-L R R705
+L R R22
 U 1 1 523E1074
 P 6500 2750
-F 0 "R705" V 6580 2750 40  0000 C CNN
+F 0 "R22" V 6580 2750 40  0000 C CNN
 F 1 "R" V 6507 2751 40  0000 C CNN
 F 2 "~" V 6430 2750 30  0000 C CNN
@@
 $EndComp
 $Comp
-L R R706
+L R R23
 U 1 1 523E107A
 P 6500 3400
-F 0 "R706" V 6580 3400 40  0000 C CNN
+F 0 "R23" V 6580 3400 40  0000 C CNN
 F 1 "R" V 6507 3401 40  0000 C CNN
 F 2 "~" V 6430 3400 30  0000 C CNN
@@
 $EndComp
 $Comp
-L R R707
+L R R24
 U 1 1 523E114C
 P 6500 4700
-F 0 "R707" V 6580 4700 40  0000 C CNN
+F 0 "R24" V 6580 4700 40  0000 C CNN
 F 1 "R" V 6507 4701 40  0000 C CNN
 F 2 "~" V 6430 4700 30  0000 C CNN
@@
 $EndComp
 $Comp
-L R R708
+L R R25
 U 1 1 523E1152
 P 6500 5400
-F 0 "R708" V 6580 5400 40  0000 C CNN
+F 0 "R25" V 6580 5400 40  0000 C CNN
 F 1 "R" V 6507 5401 40  0000 C CNN
 F 2 "~" V 6430 5400 30  0000 C CNN
@@
 	6500 3050 9350 3050
 $Comp
-L RVAR R702
+L RVAR R19
 U 1 1 523E21E8
 P 3900 6950
-F 0 "R702" V 3980 6900 50  0000 C CNN
+F 0 "R19" V 3980 6900 50  0000 C CNN
 F 1 "RVAR" V 3820 7010 50  0000 C CNN
 F 2 "~" H 3900 6950 60  0000 C CNN
@@
 $EndComp
 $Comp
-L RVAR R703
+L RVAR R20
 U 1 1 523E21FB
 P 3950 1250
-F 0 "R703" V 4030 1200 50  0000 C CNN
+F 0 "R20" V 4030 1200 50  0000 C CNN
 F 1 "RVAR" V 3870 1310 50  0000 C CNN
 F 2 "~" H 3950 1250 60  0000 C CNN
