File: BenchBudEE/Fan.sch (KiCad schematic (older format))
At the start: 9 parts

Commit message: syncing to https://github.com/ContextualElectronics/BenchBudEE/tree/ebd662c68b928f78643cdf924dc35a4d91f03121
Parts:
- removed D?: DIODE, ~, symbol DIODE
- removed Q? (x3): MOSFET_N, ~, symbol MOSFET_N
- removed R? (x2): R, ~, symbol R
- removed TH?: THERMISTOR, ~, symbol THERMISTOR
- removed U?: LM324, symbol LM324
- removed U?: MCP4921-E/MS, MSOP8, symbol MCP4921-E/MS
- added D?: DIODE, ~, symbol DIODE
- added Q? (x3): MOSFET_N, ~, symbol MOSFET_N
- added R? (x2): R, ~, symbol R
- added TH?: THERMISTOR, ~, symbol THERMISTOR
- added U?: LM324, symbol LM324
- added U?: MCP4922-E/P, DIP14, symbol MCP4922-E/P
Connections:
- net labels added: +12C, +12V, -12V
- net labels removed: -12V_FILTERED, 12V_FILTERED, 12V_FUSED
- wire segments 34 -> 45

Commit message: playing with the layout
Parts:
- gave numbers to parts that had none: 9
Changed lines of the file:
@@
-EESchema Schematic File Version 2  date 10/10/2013 12:18:22 AM
+EESchema Schematic File Version 2
 LIBS:power
 LIBS:device
@@
 Sheet 4 9
 Title ""
-Date "10 oct 2013"
+Date "3 mar 2014"
 Rev ""
 Comp ""
@@
 FAN_PWM
 $Comp
-L LM324 U?
+L LM324 U402
 U 1 1 52369784
 P 6250 3100
-F 0 "U?" H 6300 3300 60  0000 C CNN
+F 0 "U402" H 6300 3300 60  0000 C CNN
 F 1 "LM324" H 6400 2900 50  0000 C CNN
 F 2 "" H 6250 3100 60  0000 C CNN
@@
 $EndComp
 $Comp
-L MOSFET_N Q?
+L MOSFET_N Q403
 U 1 1 523697B6
 P 7800 3100
-F 0 "Q?" H 7810 3270 60  0000 R CNN
+F 0 "Q403" H 7810 3270 60  0000 R CNN
 F 1 "MOSFET_N" H 7810 2950 60  0000 R CNN
 F 2 "~" H 7800 3100 60  0000 C CNN
@@
 $EndComp
 $Comp
-L R R?
+L R R402
 U 1 1 523697E7
 P 7900 4950
-F 0 "R?" V 7980 4950 40  0000 C CNN
+F 0 "R402" V 7980 4950 40  0000 C CNN
 F 1 "R" V 7907 4951 40  0000 C CNN
 F 2 "~" V 7830 4950 30  0000 C CNN
@@
 $EndComp
 $Comp
-L AGND #PWR?
+L AGND #PWR025
 U 1 1 523697F6
 P 7900 5550
-F 0 "#PWR?" H 7900 5550 40  0001 C CNN
+F 0 "#PWR025" H 7900 5550 40  0001 C CNN
 F 1 "AGND" H 7900 5480 50  0000 C CNN
 F 2 "" H 7900 5550 60  0000 C CNN
@@
 $EndComp
 $Comp
-L +12V #PWR?
+L +12V #PWR026
 U 1 1 5236981B
 P 6150 2500
-F 0 "#PWR?" H 6150 2450 20  0001 C CNN
+F 0 "#PWR026" H 6150 2450 20  0001 C CNN
 F 1 "+12V" H 6150 2600 30  0000 C CNN
 F 2 "" H 6150 2500 60  0000 C CNN
@@
 $EndComp
 $Comp
-L -12V #PWR?
+L -12V #PWR027
 U 1 1 5236982E
 P 6150 3700
-F 0 "#PWR?" H 6150 3830 20  0001 C CNN
+F 0 "#PWR027" H 6150 3830 20  0001 C CNN
 F 1 "-12V" H 6150 3800 30  0000 C CNN
 F 2 "" H 6150 3700 60  0000 C CNN
@@
 $EndComp
 $Comp
-L AGND #PWR?
+L AGND #PWR028
 U 1 1 523698EE
 P 4700 3750
-F 0 "#PWR?" H 4700 3750 40  0001 C CNN
+F 0 "#PWR028" H 4700 3750 40  0001 C CNN
 F 1 "AGND" H 4700 3680 50  0000 C CNN
 F 2 "" H 4700 3750 60  0000 C CNN
@@
 $EndComp
 $Comp
-L MCP4922-E/P U?
+L MCP4922-E/P U401
 U 1 1 52369914
 P 2050 3150
-F 0 "U?" H 2200 3550 40  0000 L BNN
+F 0 "U401" H 2200 3550 40  0000 L BNN
 F 1 "MCP4922-E/P" H 2200 3500 40  0000 L BNN
 F 2 "DIP14" H 2050 3150 30  0000 C CIN
@@
 CURR_MEAS
 $Comp
-L R R?
+L R R401
 U 1 1 52369992
 P 3300 3000
-F 0 "R?" V 3380 3000 40  0000 C CNN
+F 0 "R401" V 3380 3000 40  0000 C CNN
 F 1 "R" V 3307 3001 40  0000 C CNN
 F 2 "~" V 3230 3000 30  0000 C CNN
@@
 SCLK
 $Comp
-L MOSFET_N Q?
+L MOSFET_N Q402
 U 1 1 5243896F
 P 7400 4950
-F 0 "Q?" H 7410 5120 60  0000 R CNN
+F 0 "Q402" H 7410 5120 60  0000 R CNN
 F 1 "MOSFET_N" H 7410 4800 60  0000 R CNN
 F 2 "~" H 7400 4950 60  0000 C CNN
@@
 $EndComp
 $Comp
-L THERMISTOR TH?
+L THERMISTOR TH401
 U 1 1 5243899F
 P 7900 1400
-F 0 "TH?" V 8000 1450 50  0000 C CNN
+F 0 "TH401" V 8000 1450 50  0000 C CNN
 F 1 "THERMISTOR" V 7800 1400 50  0000 C CNN
 F 2 "~" H 7900 1400 60  0000 C CNN
@@
 $EndComp
 $Comp
-L DIODE D?
+L DIODE D401
 U 1 1 52438A1C
 P 7450 2050
-F 0 "D?" H 7450 2150 40  0000 C CNN
+F 0 "D401" H 7450 2150 40  0000 C CNN
 F 1 "DIODE" H 7450 1950 40  0000 C CNN
 F 2 "~" H 7450 2050 60  0000 C CNN
@@
 $EndComp
 $Comp
-L MOSFET_N Q?
+L MOSFET_N Q401
 U 1 1 52438CB2
 P 4600 3400
-F 0 "Q?" H 4610 3570 60  0000 R CNN
+F 0 "Q401" H 4610 3570 60  0000 R CNN
 F 1 "MOSFET_N" H 4610 3250 60  0000 R CNN
 F 2 "~" H 4600 3400 60  0000 C CNN
@@
 	7600 3100 6750 3100
 Wire Wire Line
-	7900 3300 7900 4300
-Wire Wire Line
-	7900 4300 7900 4500
-Wire Wire Line
-	7900 4500 7900 4600
-Wire Wire Line
-	7900 4600 7900 4700
-Wire Wire Line
-	7900 5200 7900 5300
-Wire Wire Line
-	7900 5300 7900 5550
+	7900 3300 7900 4700
+Wire Wire Line
+	7900 5200 7900 5550
 Wire Wire Line
 	5350 4300 5350 3200
@@
 	6150 3700 6150 3500
 Wire Wire Line
-	3550 3000 4700 3000
-Wire Wire Line
-	4700 3000 5750 3000
+	3550 3000 5750 3000
 Wire Wire Line
 	4700 3600 4700 3750
 Wire Wire Line
-	7900 4500 1650 4500
-Wire Wire Line
-	1650 4500 1450 4500
+	1450 4500 7900 4500
 Connection ~ 7900 4500
 Wire Wire Line
-	1400 4150 1500 4150
-Wire Wire Line
-	1500 4150 3300 4150
+	1400 4150 3300 4150
 Wire Wire Line
 	2600 3000 3050 3000
@@
 	7900 1000 7900 1150
 Wire Wire Line
-	7900 1650 7900 1700
-Wire Wire Line
-	7900 1700 7900 1950
+	7900 1650 7900 1950
 Wire Wire Line
 	7900 1950 10450 1950
@@
 	10450 2200 7900 2200
 Wire Wire Line
-	7900 2200 7900 2350
-Wire Wire Line
-	7900 2350 7900 2900
+	7900 2200 7900 2900
 Wire Wire Line
 	7900 2350 7450 2350
@@
 Connection ~ 7900 5300
 Wire Wire Line
-	1700 6550 10700 6550
-Wire Wire Line
-	1700 6550 1550 6550
+	1550 6550 10700 6550
 Wire Wire Line
 	4400 3400 3300 3400
@@
 FAN_MODE
 $Comp
-L +12C #PWR?
+L +12C #PWR029
 U 1 1 5243907A
 P 7900 1000
-F 0 "#PWR?" H 7900 970 30  0001 C CNN
+F 0 "#PWR029" H 7900 970 30  0001 C CNN
 F 1 "+12C" H 7900 1110 40  0000 C CNN
 F 2 "~" H 7900 1000 60  0000 C CNN
