File: BenchBudEE/Arduino.sch (KiCad schematic (older format))
At the start: 15 parts

Commit message: syncing to https://github.com/ContextualElectronics/BenchBudEE/tree/ebd662c68b928f78643cdf924dc35a4d91f03121
Parts:
- removed ARD?: ARDUINO, ~, symbol ARDUINO
- removed R? (x14): R, ~, symbol R
- added ARD?: ARDUINOPINS, ~, symbol ARDUINOPINS
- added R? (x18): R, ~, symbol R
Connections:
- net labels added: +12P, +5V
- net labels removed: 12V_FILTERED
- wire segments 35 -> 41
Other:
- note added: "The signal Digital5 was skipped so the pin numbers for all the following pins are off by one."

Commit message: playing with the layout
Parts:
- gave numbers to parts that had none: 19
Changed lines of the file:
@@
-EESchema Schematic File Version 2  date 10/10/2013 12:18:22 AM
+EESchema Schematic File Version 2
 LIBS:power
 LIBS:device
@@
 Sheet 9 9
 Title ""
-Date "10 oct 2013"
+Date "3 mar 2014"
 Rev ""
 Comp ""
@@
 CURR_MEAS
 $Comp
-L R R?
+L R R912
 U 1 1 52400F4A
 P 6650 3900
-F 0 "R?" V 6730 3900 40  0000 C CNN
+F 0 "R912" V 6730 3900 40  0000 C CNN
 F 1 "R" V 6657 3901 40  0000 C CNN
 F 2 "~" V 6580 3900 30  0000 C CNN
@@
 	6400 3900 6050 3900
 $Comp
-L R R?
+L R R916
 U 1 1 52400F79
 P 6650 5700
-F 0 "R?" V 6730 5700 40  0000 C CNN
+F 0 "R916" V 6730 5700 40  0000 C CNN
 F 1 "R" V 6657 5701 40  0000 C CNN
 F 2 "~" V 6580 5700 30  0000 C CNN
@@
 	8500 5700 8500 6100
 $Comp
-L GND #PWR?
+L GND #PWR049
 U 1 1 524020EC
 P 8500 6100
-F 0 "#PWR?" H 8500 6100 30  0001 C CNN
+F 0 "#PWR049" H 8500 6100 30  0001 C CNN
 F 1 "GND" H 8500 6030 30  0001 C CNN
 F 2 "~" H 8500 6100 60  0000 C CNN
@@
 $EndComp
 $Comp
-L R R?
+L R R907
 U 1 1 52402349
 P 3100 5250
-F 0 "R?" V 3180 5250 40  0000 C CNN
+F 0 "R907" V 3180 5250 40  0000 C CNN
 F 1 "R" V 3107 5251 40  0000 C CNN
 F 2 "~" V 3030 5250 30  0000 C CNN
@@
 $EndComp
 $Comp
-L R R?
+L R R908
 U 1 1 5240234F
 P 3100 5450
-F 0 "R?" V 3180 5450 40  0000 C CNN
+F 0 "R908" V 3180 5450 40  0000 C CNN
 F 1 "R" V 3107 5451 40  0000 C CNN
 F 2 "~" V 3030 5450 30  0000 C CNN
@@
 V-_ADJ_MON
 $Comp
-L R R?
+L R R906
 U 1 1 52402CCD
 P 3100 5050
-F 0 "R?" V 3180 5050 40  0000 C CNN
+F 0 "R906" V 3180 5050 40  0000 C CNN
 F 1 "R" V 3107 5051 40  0000 C CNN
 F 2 "~" V 3030 5050 30  0000 C CNN
@@
 	2850 5050 2350 5050
 $Comp
-L R R?
+L R R905
 U 1 1 52402D06
 P 3100 4850
-F 0 "R?" V 3180 4850 40  0000 C CNN
+F 0 "R905" V 3180 4850 40  0000 C CNN
 F 1 "R" V 3107 4851 40  0000 C CNN
 F 2 "~" V 3030 4850 30  0000 C CNN
@@
 	3350 4850 3850 4850
 $Comp
-L R R?
+L R R909
 U 1 1 52402D2F
 P 6650 3300
-F 0 "R?" V 6730 3300 40  0000 C CNN
+F 0 "R909" V 6730 3300 40  0000 C CNN
 F 1 "R" V 6657 3301 40  0000 C CNN
 F 2 "~" V 6580 3300 30  0000 C CNN
@@
 $EndComp
 $Comp
-L R R?
+L R R910
 U 1 1 52402D35
 P 6650 3500
-F 0 "R?" V 6730 3500 40  0000 C CNN
+F 0 "R910" V 6730 3500 40  0000 C CNN
 F 1 "R" V 6657 3501 40  0000 C CNN
 F 2 "~" V 6580 3500 30  0000 C CNN
@@
 $EndComp
 $Comp
-L R R?
+L R R911
 U 1 1 52402D3B
 P 6650 3700
-F 0 "R?" V 6730 3700 40  0000 C CNN
+F 0 "R911" V 6730 3700 40  0000 C CNN
 F 1 "R" V 6657 3701 40  0000 C CNN
 F 2 "~" V 6580 3700 30  0000 C CNN
@@
 $EndComp
 $Comp
-L R R?
+L R R915
 U 1 1 52402D41
 P 6650 4500
-F 0 "R?" V 6730 4500 40  0000 C CNN
+F 0 "R915" V 6730 4500 40  0000 C CNN
 F 1 "R" V 6657 4501 40  0000 C CNN
 F 2 "~" V 6580 4500 30  0000 C CNN
@@
 	6400 4500 6050 4500
 $Comp
-L R R?
+L R R918
 U 1 1 52402DDB
 P 8900 5700
-F 0 "R?" V 8980 5700 40  0000 C CNN
+F 0 "R918" V 8980 5700 40  0000 C CNN
 F 1 "R" V 8907 5701 40  0000 C CNN
 F 2 "~" V 8830 5700 30  0000 C CNN
@@
 LED_EN_PWM
 $Comp
-L R R?
+L R R913
 U 1 1 52402E11
 P 6650 4100
-F 0 "R?" V 6730 4100 40  0000 C CNN
+F 0 "R913" V 6730 4100 40  0000 C CNN
 F 1 "R" V 6657 4101 40  0000 C CNN
 F 2 "~" V 6580 4100 30  0000 C CNN
@@
 	6400 4100 6050 4100
 $Comp
-L R R?
+L R R914
 U 1 1 5240769E
 P 6650 4300
-F 0 "R?" V 6730 4300 40  0000 C CNN
+F 0 "R914" V 6730 4300 40  0000 C CNN
 F 1 "R" V 6657 4301 40  0000 C CNN
 F 2 "~" V 6580 4300 30  0000 C CNN
@@
 FAN_MODE
 $Comp
-L R R?
+L R R917
 U 1 1 5243CF0D
 P 6650 5900
-F 0 "R?" V 6730 5900 40  0000 C CNN
+F 0 "R917" V 6730 5900 40  0000 C CNN
 F 1 "R" V 6657 5901 40  0000 C CNN
 F 2 "~" V 6580 5900 30  0000 C CNN
@@
 	6400 5900 6050 5900
 $Comp
-L R R?
+L R R904
 U 1 1 5243CF86
 P 3100 4350
-F 0 "R?" V 3180 4350 40  0000 C CNN
+F 0 "R904" V 3180 4350 40  0000 C CNN
 F 1 "R" V 3107 4351 40  0000 C CNN
 F 2 "~" V 3030 4350 30  0000 C CNN
@@
 	3350 4350 3850 4350
 $Comp
-L +12P #PWR?
+L +12P #PWR050
 U 1 1 5243CFCD
 P 1200 4050
-F 0 "#PWR?" H 1200 4020 30  0001 C CNN
+F 0 "#PWR050" H 1200 4020 30  0001 C CNN
 F 1 "+12P" H 1200 4150 30  0000 C CNN
 F 2 "~" H 1200 4050 60  0000 C CNN
@@
 	1200 4350 2850 4350
 $Comp
-L R R?
+L R R901
 U 1 1 5245171E
 P 3100 3750
-F 0 "R?" V 3180 3750 40  0000 C CNN
+F 0 "R901" V 3180 3750 40  0000 C CNN
 F 1 "R" V 3107 3751 40  0000 C CNN
 F 2 "~" V 3030 3750 30  0000 C CNN
@@
 	3350 3750 3850 3750
 $Comp
-L +5V #PWR?
+L +5V #PWR051
 U 1 1 5245176C
 P 1200 3500
-F 0 "#PWR?" H 1200 3590 20  0001 C CNN
+F 0 "#PWR051" H 1200 3590 20  0001 C CNN
 F 1 "+5V" H 1200 3590 30  0000 C CNN
 F 2 "~" H 1200 3500 60  0000 C CNN
@@
 	3850 3950 3350 3950
 $Comp
-L R R?
+L R R902
 U 1 1 524517C0
 P 3100 3950
-F 0 "R?" V 3180 3950 40  0000 C CNN
+F 0 "R902" V 3180 3950 40  0000 C CNN
 F 1 "R" V 3107 3951 40  0000 C CNN
 F 2 "~" V 3030 3950 30  0000 C CNN
@@
 $EndComp
 $Comp
-L R R?
+L R R903
 U 1 1 524517C6
 P 3100 4150
-F 0 "R?" V 3180 4150 40  0000 C CNN
+F 0 "R903" V 3180 4150 40  0000 C CNN
 F 1 "R" V 3107 4151 40  0000 C CNN
 F 2 "~" V 3030 4150 30  0000 C CNN
@@
 	2100 3950 2100 4150
 $Comp
-L GND #PWR?
+L GND #PWR052
 U 1 1 5245181B
 P 2100 4150
-F 0 "#PWR?" H 2100 4150 30  0001 C CNN
+F 0 "#PWR052" H 2100 4150 30  0001 C CNN
 F 1 "GND" H 2100 4080 30  0001 C CNN
 F 2 "~" H 2100 4150 60  0000 C CNN
@@
 The signal Digital5 was skipped so the pin numbers for all the following pins are off by one.
 $Comp
-L ARDUINOPINS ARD?
+L ARDUINOPINS ARD901
 U 1 1 5251D4C8
 P 4950 4450
-F 0 "ARD?" H 4300 6050 60  0000 C CNN
+F 0 "ARD901" H 4300 6050 60  0000 C CNN
 F 1 "ARDUINOPINS" H 4450 6250 60  0000 C CNN
 F 2 "~" H 5500 3500 60  0000 C CNN

Commit message: syncing to upstream
Parts:
- renumbered ARD901 to ARD1, R901 to R26, R902 to R27, R903 to R28, R904 to R29, R905 to R30, R906 to R31, R907 to R32, R908 to R33, R909 to R34, R910 to R35, R911 to R36, R912 to R37, R913 to R38, R914 to R39, R915 to R40, R916 to R41, R917 to R42, R918 to R43
Changed lines of the file:
@@
-EESchema Schematic File Version 2
+EESchema Schematic File Version 2  date 10/10/2013 1:06:29 AM
 LIBS:power
 LIBS:device
@@
 Sheet 9 9
 Title ""
-Date "3 mar 2014"
+Date "10 oct 2013"
 Rev ""
 Comp ""
@@
 CURR_MEAS
 $Comp
-L R R912
+L R R37
 U 1 1 52400F4A
 P 6650 3900
-F 0 "R912" V 6730 3900 40  0000 C CNN
+F 0 "R37" V 6730 3900 40  0000 C CNN
 F 1 "R" V 6657 3901 40  0000 C CNN
 F 2 "~" V 6580 3900 30  0000 C CNN
@@
 	6400 3900 6050 3900
 $Comp
-L R R916
+L R R41
 U 1 1 52400F79
 P 6650 5700
-F 0 "R916" V 6730 5700 40  0000 C CNN
+F 0 "R41" V 6730 5700 40  0000 C CNN
 F 1 "R" V 6657 5701 40  0000 C CNN
 F 2 "~" V 6580 5700 30  0000 C CNN
@@
 	8500 5700 8500 6100
 $Comp
-L GND #PWR049
+L GND #PWR55
 U 1 1 524020EC
 P 8500 6100
-F 0 "#PWR049" H 8500 6100 30  0001 C CNN
+F 0 "#PWR55" H 8500 6100 30  0001 C CNN
 F 1 "GND" H 8500 6030 30  0001 C CNN
 F 2 "~" H 8500 6100 60  0000 C CNN
@@
 $EndComp
 $Comp
-L R R907
+L R R32
 U 1 1 52402349
 P 3100 5250
-F 0 "R907" V 3180 5250 40  0000 C CNN
+F 0 "R32" V 3180 5250 40  0000 C CNN
 F 1 "R" V 3107 5251 40  0000 C CNN
 F 2 "~" V 3030 5250 30  0000 C CNN
@@
 $EndComp
 $Comp
-L R R908
+L R R33
 U 1 1 5240234F
 P 3100 5450
-F 0 "R908" V 3180 5450 40  0000 C CNN
+F 0 "R33" V 3180 5450 40  0000 C CNN
 F 1 "R" V 3107 5451 40  0000 C CNN
 F 2 "~" V 3030 5450 30  0000 C CNN
@@
 V-_ADJ_MON
 $Comp
-L R R906
+L R R31
 U 1 1 52402CCD
 P 3100 5050
-F 0 "R906" V 3180 5050 40  0000 C CNN
+F 0 "R31" V 3180 5050 40  0000 C CNN
 F 1 "R" V 3107 5051 40  0000 C CNN
 F 2 "~" V 3030 5050 30  0000 C CNN
@@
 	2850 5050 2350 5050
 $Comp
-L R R905
+L R R30
 U 1 1 52402D06
 P 3100 4850
-F 0 "R905" V 3180 4850 40  0000 C CNN
+F 0 "R30" V 3180 4850 40  0000 C CNN
 F 1 "R" V 3107 4851 40  0000 C CNN
 F 2 "~" V 3030 4850 30  0000 C CNN
@@
 	3350 4850 3850 4850
 $Comp
-L R R909
+L R R34
 U 1 1 52402D2F
 P 6650 3300
-F 0 "R909" V 6730 3300 40  0000 C CNN
+F 0 "R34" V 6730 3300 40  0000 C CNN
 F 1 "R" V 6657 3301 40  0000 C CNN
 F 2 "~" V 6580 3300 30  0000 C CNN
@@
 $EndComp
 $Comp
-L R R910
+L R R35
 U 1 1 52402D35
 P 6650 3500
-F 0 "R910" V 6730 3500 40  0000 C CNN
+F 0 "R35" V 6730 3500 40  0000 C CNN
 F 1 "R" V 6657 3501 40  0000 C CNN
 F 2 "~" V 6580 3500 30  0000 C CNN
@@
 $EndComp
 $Comp
-L R R911
+L R R36
 U 1 1 52402D3B
 P 6650 3700
-F 0 "R911" V 6730 3700 40  0000 C CNN
+F 0 "R36" V 6730 3700 40  0000 C CNN
 F 1 "R" V 6657 3701 40  0000 C CNN
 F 2 "~" V 6580 3700 30  0000 C CNN
@@
 $EndComp
 $Comp
-L R R915
+L R R40
 U 1 1 52402D41
 P 6650 4500
-F 0 "R915" V 6730 4500 40  0000 C CNN
+F 0 "R40" V 6730 4500 40  0000 C CNN
 F 1 "R" V 6657 4501 40  0000 C CNN
 F 2 "~" V 6580 4500 30  0000 C CNN
@@
 	6400 4500 6050 4500
 $Comp
-L R R918
+L R R43
 U 1 1 52402DDB
 P 8900 5700
-F 0 "R918" V 8980 5700 40  0000 C CNN
+F 0 "R43" V 8980 5700 40  0000 C CNN
 F 1 "R" V 8907 5701 40  0000 C CNN
 F 2 "~" V 8830 5700 30  0000 C CNN
@@
 LED_EN_PWM
 $Comp
-L R R913
+L R R38
 U 1 1 52402E11
 P 6650 4100
-F 0 "R913" V 6730 4100 40  0000 C CNN
+F 0 "R38" V 6730 4100 40  0000 C CNN
 F 1 "R" V 6657 4101 40  0000 C CNN
 F 2 "~" V 6580 4100 30  0000 C CNN
@@
 	6400 4100 6050 4100
 $Comp
-L R R914
+L R R39
 U 1 1 5240769E
 P 6650 4300
-F 0 "R914" V 6730 4300 40  0000 C CNN
+F 0 "R39" V 6730 4300 40  0000 C CNN
 F 1 "R" V 6657 4301 40  0000 C CNN
 F 2 "~" V 6580 4300 30  0000 C CNN
@@
 FAN_MODE
 $Comp
-L R R917
+L R R42
 U 1 1 5243CF0D
 P 6650 5900
-F 0 "R917" V 6730 5900 40  0000 C CNN
+F 0 "R42" V 6730 5900 40  0000 C CNN
 F 1 "R" V 6657 5901 40  0000 C CNN
 F 2 "~" V 6580 5900 30  0000 C CNN
@@
 	6400 5900 6050 5900
 $Comp
-L R R904
+L R R29
 U 1 1 5243CF86
 P 3100 4350
-F 0 "R904" V 3180 4350 40  0000 C CNN
+F 0 "R29" V 3180 4350 40  0000 C CNN
 F 1 "R" V 3107 4351 40  0000 C CNN
 F 2 "~" V 3030 4350 30  0000 C CNN
@@
 	3350 4350 3850 4350
 $Comp
-L +12P #PWR050
+L +12P #PWR53
 U 1 1 5243CFCD
 P 1200 4050
-F 0 "#PWR050" H 1200 4020 30  0001 C CNN
+F 0 "#PWR53" H 1200 4020 30  0001 C CNN
 F 1 "+12P" H 1200 4150 30  0000 C CNN
 F 2 "~" H 1200 4050 60  0000 C CNN
@@
 	1200 4350 2850 4350
 $Comp
-L R R901
+L R R26
 U 1 1 5245171E
 P 3100 3750
-F 0 "R901" V 3180 3750 40  0000 C CNN
+F 0 "R26" V 3180 3750 40  0000 C CNN
 F 1 "R" V 3107 3751 40  0000 C CNN
 F 2 "~" V 3030 3750 30  0000 C CNN
@@
 	3350 3750 3850 3750
 $Comp
-L +5V #PWR051
+L +5V #PWR52
 U 1 1 5245176C
 P 1200 3500
-F 0 "#PWR051" H 1200 3590 20  0001 C CNN
+F 0 "#PWR52" H 1200 3590 20  0001 C CNN
 F 1 "+5V" H 1200 3590 30  0000 C CNN
 F 2 "~" H 1200 3500 60  0000 C CNN
@@
 	3850 3950 3350 3950
 $Comp
-L R R902
+L R R27
 U 1 1 524517C0
 P 3100 3950
-F 0 "R902" V 3180 3950 40  0000 C CNN
+F 0 "R27" V 3180 3950 40  0000 C CNN
 F 1 "R" V 3107 3951 40  0000 C CNN
 F 2 "~" V 3030 3950 30  0000 C CNN
@@
 $EndComp
 $Comp
-L R R903
+L R R28
 U 1 1 524517C6
 P 3100 4150
-F 0 "R903" V 3180 4150 40  0000 C CNN
+F 0 "R28" V 3180 4150 40  0000 C CNN
 F 1 "R" V 3107 4151 40  0000 C CNN
 F 2 "~" V 3030 4150 30  0000 C CNN
@@
 	2100 3950 2100 4150
 $Comp
-L GND #PWR052
+L GND #PWR54
 U 1 1 5245181B
 P 2100 4150
-F 0 "#PWR052" H 2100 4150 30  0001 C CNN
+F 0 "#PWR54" H 2100 4150 30  0001 C CNN
 F 1 "GND" H 2100 4080 30  0001 C CNN
 F 2 "~" H 2100 4150 60  0000 C CNN
@@
 The signal Digital5 was skipped so the pin numbers for all the following pins are off by one.
 $Comp
-L ARDUINOPINS ARD901
+L ARDUINOPINS ARD1
 U 1 1 5251D4C8
 P 4950 4450
-F 0 "ARD901" H 4300 6050 60  0000 C CNN
+F 0 "ARD1" H 4300 6050 60  0000 C CNN
 F 1 "ARDUINOPINS" H 4450 6250 60  0000 C CNN
 F 2 "~" H 5500 3500 60  0000 C CNN
