File: BenchBudEE/LED_Driver.sch (KiCad schematic (older format))
At the start: 6 parts

Commit message: playing with the layout
Parts:
- gave numbers to parts that had none: 6
Changed lines of the file:
@@
-EESchema Schematic File Version 2  date 10/10/2013 12:18:22 AM
+EESchema Schematic File Version 2
 LIBS:power
 LIBS:device
@@
 Sheet 6 9
 Title ""
-Date "10 oct 2013"
+Date "3 mar 2014"
 Rev ""
 Comp ""
@@
 LED_STRING+
 $Comp
-L AP5726 U?
+L AP5726 U501
 U 1 1 523F52C8
 P 3650 3050
-F 0 "U?" H 4000 2400 60  0000 C CNN
+F 0 "U501" H 4000 2400 60  0000 C CNN
 F 1 "AP5726" H 3650 3050 60  0000 C CNN
 F 2 "" H 3550 3150 60  0000 C CNN
@@
 	2150 2950 2850 2950
 $Comp
-L +5V #PWR?
+L +5V #PWR030
 U 1 1 523F5D4A
 P 2550 1450
-F 0 "#PWR?" H 2550 1540 20  0001 C CNN
+F 0 "#PWR030" H 2550 1540 20  0001 C CNN
 F 1 "+5V" H 2550 1540 30  0000 C CNN
 F 2 "~" H 2550 1450 60  0000 C CNN
@@
 $EndComp
 $Comp
-L GND #PWR?
+L GND #PWR031
 U 1 1 523F5D68
 P 2550 2350
-F 0 "#PWR?" H 2550 2350 30  0001 C CNN
+F 0 "#PWR031" H 2550 2350 30  0001 C CNN
 F 1 "GND" H 2550 2280 30  0001 C CNN
 F 2 "~" H 2550 2350 60  0000 C CNN
@@
 $EndComp
 $Comp
-L GND #PWR?
+L GND #PWR032
 U 1 1 523F5D75
 P 3650 4150
-F 0 "#PWR?" H 3650 4150 30  0001 C CNN
+F 0 "#PWR032" H 3650 4150 30  0001 C CNN
 F 1 "GND" H 3650 4080 30  0001 C CNN
 F 2 "~" H 3650 4150 60  0000 C CNN
@@
 	3650 4150 3650 3900
 $Comp
-L C C?
+L C C501
 U 1 1 523F5D89
 P 2550 1950
-F 0 "C?" H 2550 2050 40  0000 L CNN
+F 0 "C501" H 2550 2050 40  0000 L CNN
 F 1 "C" H 2556 1865 40  0000 L CNN
 F 2 "~" H 2588 1800 30  0000 C CNN
@@
 Connection ~ 2550 1650
 $Comp
-L C C?
+L C C502
 U 1 1 523F5DA2
 P 9400 2100
-F 0 "C?" H 9400 2200 40  0000 L CNN
+F 0 "C502" H 9400 2200 40  0000 L CNN
 F 1 "C" H 9406 2015 40  0000 L CNN
 F 2 "~" H 9438 1950 30  0000 C CNN
@@
 $EndComp
 $Comp
-L INDUCTOR L?
+L INDUCTOR L501
 U 1 1 523F5DAA
 P 3950 1650
-F 0 "L?" V 3900 1650 40  0000 C CNN
+F 0 "L501" V 3900 1650 40  0000 C CNN
 F 1 "INDUCTOR" V 4050 1650 40  0000 C CNN
 F 2 "~" H 3950 1650 60  0000 C CNN
@@
 	4250 1650 4750 1650
 $Comp
-L DIODESCH D?
+L DIODESCH D501
 U 1 1 523F5DF0
 P 4950 1650
-F 0 "D?" H 4950 1750 40  0000 C CNN
+F 0 "D501" H 4950 1750 40  0000 C CNN
 F 1 "DIODESCH" H 4950 1550 40  0000 C CNN
 F 2 "~" H 4950 1650 60  0000 C CNN
@@
 	9400 1650 9400 1900
 $Comp
-L GND #PWR?
+L GND #PWR033
 U 1 1 523F5E22
 P 9400 2450
-F 0 "#PWR?" H 9400 2450 30  0001 C CNN
+F 0 "#PWR033" H 9400 2450 30  0001 C CNN
 F 1 "GND" H 9400 2380 30  0001 C CNN
 F 2 "~" H 9400 2450 60  0000 C CNN
@@
 Connection ~ 9400 1650
 $Comp
-L R R?
+L R R501
 U 1 1 523F5E65
 P 4800 3600
-F 0 "R?" V 4880 3600 40  0000 C CNN
+F 0 "R501" V 4880 3600 40  0000 C CNN
 F 1 "R" V 4807 3601 40  0000 C CNN
 F 2 "~" V 4730 3600 30  0000 C CNN

Commit message: syncing to upstream
Parts:
- renumbered C501 to C5, C502 to C6, D501 to D5, L501 to L4, R501 to R17, U501 to U7
Changed lines of the file:
@@
-EESchema Schematic File Version 2
+EESchema Schematic File Version 2  date 10/10/2013 1:06:29 AM
 LIBS:power
 LIBS:device
@@
 Sheet 6 9
 Title ""
-Date "3 mar 2014"
+Date "10 oct 2013"
 Rev ""
 Comp ""
@@
 LED_STRING+
 $Comp
-L AP5726 U501
+L AP5726 U7
 U 1 1 523F52C8
 P 3650 3050
-F 0 "U501" H 4000 2400 60  0000 C CNN
+F 0 "U7" H 4000 2400 60  0000 C CNN
 F 1 "AP5726" H 3650 3050 60  0000 C CNN
 F 2 "" H 3550 3150 60  0000 C CNN
@@
 	2150 2950 2850 2950
 $Comp
-L +5V #PWR030
+L +5V #PWR32
 U 1 1 523F5D4A
 P 2550 1450
-F 0 "#PWR030" H 2550 1540 20  0001 C CNN
+F 0 "#PWR32" H 2550 1540 20  0001 C CNN
 F 1 "+5V" H 2550 1540 30  0000 C CNN
 F 2 "~" H 2550 1450 60  0000 C CNN
@@
 $EndComp
 $Comp
-L GND #PWR031
+L GND #PWR33
 U 1 1 523F5D68
 P 2550 2350
-F 0 "#PWR031" H 2550 2350 30  0001 C CNN
+F 0 "#PWR33" H 2550 2350 30  0001 C CNN
 F 1 "GND" H 2550 2280 30  0001 C CNN
 F 2 "~" H 2550 2350 60  0000 C CNN
@@
 $EndComp
 $Comp
-L GND #PWR032
+L GND #PWR34
 U 1 1 523F5D75
 P 3650 4150
-F 0 "#PWR032" H 3650 4150 30  0001 C CNN
+F 0 "#PWR34" H 3650 4150 30  0001 C CNN
 F 1 "GND" H 3650 4080 30  0001 C CNN
 F 2 "~" H 3650 4150 60  0000 C CNN
@@
 	3650 4150 3650 3900
 $Comp
-L C C501
+L C C5
 U 1 1 523F5D89
 P 2550 1950
-F 0 "C501" H 2550 2050 40  0000 L CNN
+F 0 "C5" H 2550 2050 40  0000 L CNN
 F 1 "C" H 2556 1865 40  0000 L CNN
 F 2 "~" H 2588 1800 30  0000 C CNN
@@
 Connection ~ 2550 1650
 $Comp
-L C C502
+L C C6
 U 1 1 523F5DA2
 P 9400 2100
-F 0 "C502" H 9400 2200 40  0000 L CNN
+F 0 "C6" H 9400 2200 40  0000 L CNN
 F 1 "C" H 9406 2015 40  0000 L CNN
 F 2 "~" H 9438 1950 30  0000 C CNN
@@
 $EndComp
 $Comp
-L INDUCTOR L501
+L INDUCTOR L4
 U 1 1 523F5DAA
 P 3950 1650
-F 0 "L501" V 3900 1650 40  0000 C CNN
+F 0 "L4" V 3900 1650 40  0000 C CNN
 F 1 "INDUCTOR" V 4050 1650 40  0000 C CNN
 F 2 "~" H 3950 1650 60  0000 C CNN
@@
 	4250 1650 4750 1650
 $Comp
-L DIODESCH D501
+L DIODESCH D5
 U 1 1 523F5DF0
 P 4950 1650
-F 0 "D501" H 4950 1750 40  0000 C CNN
+F 0 "D5" H 4950 1750 40  0000 C CNN
 F 1 "DIODESCH" H 4950 1550 40  0000 C CNN
 F 2 "~" H 4950 1650 60  0000 C CNN
@@
 	9400 1650 9400 1900
 $Comp
-L GND #PWR033
+L GND #PWR35
 U 1 1 523F5E22
 P 9400 2450
-F 0 "#PWR033" H 9400 2450 30  0001 C CNN
+F 0 "#PWR35" H 9400 2450 30  0001 C CNN
 F 1 "GND" H 9400 2380 30  0001 C CNN
 F 2 "~" H 9400 2450 60  0000 C CNN
@@
 Connection ~ 9400 1650
 $Comp
-L R R501
+L R R17
 U 1 1 523F5E65
 P 4800 3600
-F 0 "R501" V 4880 3600 40  0000 C CNN
+F 0 "R17" V 4880 3600 40  0000 C CNN
 F 1 "R" V 4807 3601 40  0000 C CNN
 F 2 "~" V 4730 3600 30  0000 C CNN
