File: BenchBudEE/Thermocouple.sch (KiCad schematic (older format))
At the start: 14 parts

Commit message: syncing to https://github.com/ContextualElectronics/BenchBudEE/tree/ebd662c68b928f78643cdf924dc35a4d91f03121
Parts:
- removed D?: ZENER, ~, symbol ZENER
- removed R? (x7): R, ~, symbol R
- removed U? (x4): LM324, symbol LM324
- removed U? (x2): MCP3550-60-E/SN, SO8, symbol MCP3550-60-E/SN
- added C?: C, ~, symbol C
- added D?: ZENER, ~, symbol ZENER
- added R? (x7): R, ~, symbol R
- added U? (x4): LM324, symbol LM324
- added U? (x2): MCP3550-60-E/SN, SO8, symbol MCP3550-60-E/SN
Connections:
- net +12V: now also D?.2 (K), U?.3 (+), U?.4 (V+), U?.4 (V+), U?.4 (V+)
- net -12V: now also U?.11 (V-), U?.11 (V-), U?.11 (V-)
- net AGND: now also D?.1 (A), R?.1, U?.3 (Vin-), U?.3 (Vin-)
- net CS_N: now also U?.7 (~CS~)
- net MISO: now also U?.6 (SDO/~RDY~)
- net SCLK: now also U?.5 (SCK)
- new net: R?.1, R?.2, U?.1
- new net: R?.1, R?.2, U?.2 (-) (x3)
- new net: R?.2, R?.2, U?.1
- new net: R?.1, U?.1, U?.2 (Vin+)
- new net: R?.1, R?.2, U?.3 (+)
- new net: U?.1, U?.2 (-), U?.2 (Vin+)
- new net TC IN +: U?.3 (+)
- new net TC IN -: U?.3 (+)
Other:
- note added: "16-24Bit ADC"
- note added: "Analog/TC Input"
- note added: "General Temperature Sensor"
- note added: "Instrumentation Amp"
- note removed: "16-24 bit ADC"
- note removed: "Instrumentation Amplifier"
- note removed: "Thermocouple\nInput"
- note removed: "general temp sensor"

Commit message: playing with the layout
Parts:
- gave numbers to parts that had none: 12
Connections:
- net +12V: now also U203.5 (+); no longer U203.3 (+)
- net TC IN +: now also U203.10 (+); no longer U203.3 (+)
- net TC IN -: now also U203.12 (+); no longer U203.3 (+)
- net at R203.2, R205.1: now also U203.8; no longer U203.1
- net at R205.2, R206.1: now also U203.9 (-); no longer U203.2 (-)
- net at R204.2, R207.2: now also U203.14; no longer U203.1
- net at R206.2, R207.1: now also U203.13 (-); no longer U203.2 (-)
- new net: U202.2 (Vin+), U203.6 (-), U203.7
Changed lines of the file:
@@
-EESchema Schematic File Version 2  date 10/10/2013 12:18:22 AM
+EESchema Schematic File Version 2
 LIBS:power
 LIBS:device
@@
 Sheet 3 9
 Title ""
-Date "10 oct 2013"
+Date "3 mar 2014"
 Rev ""
 Comp ""
@@
 CS_N
 $Comp
-L LM324 U?
-U 1 1 523643C2
+L LM324 U203
+U 3 1 523643C2
 P 8900 2350
-F 0 "U?" H 8950 2550 60  0000 C CNN
+F 0 "U203" H 8950 2550 60  0000 C CNN
 F 1 "LM324" H 9050 2150 50  0000 C CNN
 F 2 "" H 8900 2350 60  0000 C CNN
 F 3 "" H 8900 2350 60  0000 C CNN
-	1    8900 2350
+	3    8900 2350
 	-1   0    0    -1
 $EndComp
 $Comp
-L LM324 U?
-U 1 1 523643CF
+L LM324 U203
+U 4 1 523643CF
 P 8900 4450
-F 0 "U?" H 8950 4650 60  0000 C CNN
+F 0 "U203" H 8950 4650 60  0000 C CNN
 F 1 "LM324" H 9050 4250 50  0000 C CNN
 F 2 "" H 8900 4450 60  0000 C CNN
 F 3 "" H 8900 4450 60  0000 C CNN
-	1    8900 4450
+	4    8900 4450
 	-1   0    0    1
 $EndComp
 $Comp
-L LM324 U?
+L LM324 U203
 U 1 1 523643D5
 P 6150 3300
-F 0 "U?" H 6200 3500 60  0000 C CNN
+F 0 "U203" H 6200 3500 60  0000 C CNN
 F 1 "LM324" H 6300 3100 50  0000 C CNN
 F 2 "" H 6150 3300 60  0000 C CNN
@@
 $EndComp
 $Comp
-L LM324 U?
-U 1 1 523643DB
+L LM324 U203
+U 2 1 523643DB
 P 8000 6100
-F 0 "U?" H 8050 6300 60  0000 C CNN
+F 0 "U203" H 8050 6300 60  0000 C CNN
 F 1 "LM324" H 8150 5900 50  0000 C CNN
 F 2 "" H 8000 6100 60  0000 C CNN
 F 3 "" H 8000 6100 60  0000 C CNN
-	1    8000 6100
+	2    8000 6100
 	-1   0    0    -1
 $EndComp
 $Comp
-L C C?
+L C C201
 U 1 1 523643FC
 P 7250 3950
-F 0 "C?" H 7250 4050 40  0000 L CNN
+F 0 "C201" H 7250 4050 40  0000 L CNN
 F 1 "C" H 7256 3865 40  0000 L CNN
 F 2 "~" H 7288 3800 30  0000 C CNN
@@
 $EndComp
 $Comp
-L R R?
+L R R205
 U 1 1 5236440B
 P 8100 2750
-F 0 "R?" V 8180 2750 40  0000 C CNN
+F 0 "R205" V 8180 2750 40  0000 C CNN
 F 1 "R" V 8107 2751 40  0000 C CNN
 F 2 "~" V 8030 2750 30  0000 C CNN
@@
 $EndComp
 $Comp
-L R R?
+L R R206
 U 1 1 52364427
 P 8100 3400
-F 0 "R?" V 8180 3400 40  0000 C CNN
+F 0 "R206" V 8180 3400 40  0000 C CNN
 F 1 "R" V 8107 3401 40  0000 C CNN
 F 2 "~" V 8030 3400 30  0000 C CNN
@@
 $EndComp
 $Comp
-L R R?
+L R R207
 U 1 1 5236442D
 P 8100 4000
-F 0 "R?" V 8180 4000 40  0000 C CNN
+F 0 "R207" V 8180 4000 40  0000 C CNN
 F 1 "R" V 8107 4001 40  0000 C CNN
 F 2 "~" V 8030 4000 30  0000 C CNN
@@
 $EndComp
 $Comp
-L R R?
+L R R203
 U 1 1 5236444F
 P 7300 2350
-F 0 "R?" V 7380 2350 40  0000 C CNN
+F 0 "R203" V 7380 2350 40  0000 C CNN
 F 1 "R" V 7307 2351 40  0000 C CNN
 F 2 "~" V 7230 2350 30  0000 C CNN
@@
 $EndComp
 $Comp
-L R R?
+L R R202
 U 1 1 52364455
 P 5400 2350
-F 0 "R?" V 5480 2350 40  0000 C CNN
+F 0 "R202" V 5480 2350 40  0000 C CNN
 F 1 "R" V 5407 2351 40  0000 C CNN
 F 2 "~" V 5330 2350 30  0000 C CNN
@@
 $EndComp
 $Comp
-L R R?
+L R R201
 U 1 1 5236445B
 P 5350 4450
-F 0 "R?" V 5430 4450 40  0000 C CNN
+F 0 "R201" V 5430 4450 40  0000 C CNN
 F 1 "R" V 5357 4451 40  0000 C CNN
 F 2 "~" V 5280 4450 30  0000 C CNN
@@
 $EndComp
 $Comp
-L R R?
+L R R204
 U 1 1 52364461
 P 7300 4450
-F 0 "R?" V 7380 4450 40  0000 C CNN
+F 0 "R204" V 7380 4450 40  0000 C CNN
 F 1 "R" V 7307 4451 40  0000 C CNN
 F 2 "~" V 7230 4450 30  0000 C CNN
@@
 $EndComp
 $Comp
-L -12V #PWR?
+L -12V #PWR01
 U 1 1 523646A5
 P 6250 2800
-F 0 "#PWR?" H 6250 2930 20  0001 C CNN
+F 0 "#PWR01" H 6250 2930 20  0001 C CNN
 F 1 "-12V" H 6250 2900 30  0000 C CNN
 F 2 "" H 6250 2800 60  0000 C CNN
@@
 $EndComp
 $Comp
-L -12V #PWR?
+L -12V #PWR02
 U 1 1 523646B2
 P 9000 2850
-F 0 "#PWR?" H 9000 2980 20  0001 C CNN
+F 0 "#PWR02" H 9000 2980 20  0001 C CNN
 F 1 "-12V" H 9000 2950 30  0000 C CNN
 F 2 "" H 9000 2850 60  0000 C CNN
@@
 $EndComp
 $Comp
-L -12V #PWR?
+L -12V #PWR03
 U 1 1 523646B8
 P 9000 3950
-F 0 "#PWR?" H 9000 4080 20  0001 C CNN
+F 0 "#PWR03" H 9000 4080 20  0001 C CNN
 F 1 "-12V" H 9000 4050 30  0000 C CNN
 F 2 "" H 9000 3950 60  0000 C CNN
@@
 $EndComp
 $Comp
-L +12V #PWR?
+L +12V #PWR04
 U 1 1 5236471D
 P 6250 3850
-F 0 "#PWR?" H 6250 3800 20  0001 C CNN
+F 0 "#PWR04" H 6250 3800 20  0001 C CNN
 F 1 "+12V" H 6250 3950 30  0000 C CNN
 F 2 "" H 6250 3850 60  0000 C CNN
@@
 $EndComp
 $Comp
-L +12V #PWR?
+L +12V #PWR05
 U 1 1 5236474B
 P 9000 1800
-F 0 "#PWR?" H 9000 1750 20  0001 C CNN
+F 0 "#PWR05" H 9000 1750 20  0001 C CNN
 F 1 "+12V" H 9000 1900 30  0000 C CNN
 F 2 "" H 9000 1800 60  0000 C CNN
@@
 $EndComp
 $Comp
-L +12V #PWR?
+L +12V #PWR06
 U 1 1 52364796
 P 9000 5000
-F 0 "#PWR?" H 9000 4950 20  0001 C CNN
+F 0 "#PWR06" H 9000 4950 20  0001 C CNN
 F 1 "+12V" H 9000 5100 30  0000 C CNN
 F 2 "" H 9000 5000 60  0000 C CNN
@@
 	9000 5000 9000 4850
 $Comp
-L AGND #PWR?
+L AGND #PWR07
 U 1 1 52364808
 P 4900 4700
-F 0 "#PWR?" H 4900 4700 40  0001 C CNN
+F 0 "#PWR07" H 4900 4700 40  0001 C CNN
 F 1 "AGND" H 4900 4630 50  0000 C CNN
 F 2 "" H 4900 4700 60  0000 C CNN
@@
 	4900 3600 4900 4700
 $Comp
-L MCP3550-60-E/SN U?
+L MCP3550-60-E/SN U201
 U 1 1 5236486B
 P 2350 3450
-F 0 "U?" H 1800 3800 40  0000 C CNN
+F 0 "U201" H 1800 3800 40  0000 C CNN
 F 1 "MCP3550-60-E/SN" H 2050 3750 40  0000 C CNN
 F 2 "SO8" H 2150 3450 30  0000 C CIN
@@
 	950  3550 1850 3550
 $Comp
-L MCP3550-60-E/SN U?
+L MCP3550-60-E/SN U202
 U 1 1 523649E1
 P 2350 6100
-F 0 "U?" H 1800 6450 40  0000 C CNN
+F 0 "U202" H 1800 6450 40  0000 C CNN
 F 1 "MCP3550-60-E/SN" H 2050 6400 40  0000 C CNN
 F 2 "SO8" H 2150 6100 30  0000 C CIN
@@
 $EndComp
 $Comp
-L ZENER D?
+L ZENER D201
 U 1 1 523649F3
 P 9700 6250
-F 0 "D?" H 9700 6350 50  0000 C CNN
+F 0 "D201" H 9700 6350 50  0000 C CNN
 F 1 "ZENER" H 9700 6150 40  0000 C CNN
 F 2 "~" H 9700 6250 60  0000 C CNN
@@
 $EndComp
 $Comp
-L +12V #PWR?
+L +12V #PWR08
 U 1 1 52364A00
 P 9700 5700
-F 0 "#PWR?" H 9700 5650 20  0001 C CNN
+F 0 "#PWR08" H 9700 5650 20  0001 C CNN
 F 1 "+12V" H 9700 5800 30  0000 C CNN
 F 2 "" H 9700 5700 60  0000 C CNN
@@
 	9700 6450 9700 6700
 $Comp
-L AGND #PWR?
+L AGND #PWR09
 U 1 1 52364A60
 P 9700 6700
-F 0 "#PWR?" H 9700 6700 40  0001 C CNN
+F 0 "#PWR09" H 9700 6700 40  0001 C CNN
 F 1 "AGND" H 9700 6630 50  0000 C CNN
 F 2 "" H 9700 6700 60  0000 C CNN
@@
 Connection ~ 7250 6100
 $Comp
-L AGND #PWR?
+L AGND #PWR010
 U 1 1 52364B5B
 P 3000 6450
-F 0 "#PWR?" H 3000 6450 40  0001 C CNN
+F 0 "#PWR010" H 3000 6450 40  0001 C CNN
 F 1 "AGND" H 3000 6380 50  0000 C CNN
 F 2 "" H 3000 6450 60  0000 C CNN

Commit message: syncing to upstream
Parts:
- renumbered C201 to C1, D201 to D3, R204 to R10, R205 to R11, R206 to R12, R207 to R13, R201 to R7, R202 to R8, R203 to R9, U201 to U2, U202 to U3, U203 to U4
Changed lines of the file:
@@
-EESchema Schematic File Version 2
+EESchema Schematic File Version 2  date 10/10/2013 1:06:29 AM
 LIBS:power
 LIBS:device
@@
 Sheet 3 9
 Title ""
-Date "3 mar 2014"
+Date "10 oct 2013"
 Rev ""
 Comp ""
@@
 CS_N
 $Comp
-L LM324 U203
+L LM324 U4
 U 3 1 523643C2
 P 8900 2350
-F 0 "U203" H 8950 2550 60  0000 C CNN
+F 0 "U4" H 8950 2550 60  0000 C CNN
 F 1 "LM324" H 9050 2150 50  0000 C CNN
 F 2 "" H 8900 2350 60  0000 C CNN
@@
 $EndComp
 $Comp
-L LM324 U203
+L LM324 U4
 U 4 1 523643CF
 P 8900 4450
-F 0 "U203" H 8950 4650 60  0000 C CNN
+F 0 "U4" H 8950 4650 60  0000 C CNN
 F 1 "LM324" H 9050 4250 50  0000 C CNN
 F 2 "" H 8900 4450 60  0000 C CNN
@@
 $EndComp
 $Comp
-L LM324 U203
+L LM324 U4
 U 1 1 523643D5
 P 6150 3300
-F 0 "U203" H 6200 3500 60  0000 C CNN
+F 0 "U4" H 6200 3500 60  0000 C CNN
 F 1 "LM324" H 6300 3100 50  0000 C CNN
 F 2 "" H 6150 3300 60  0000 C CNN
@@
 $EndComp
 $Comp
-L LM324 U203
+L LM324 U4
 U 2 1 523643DB
 P 8000 6100
-F 0 "U203" H 8050 6300 60  0000 C CNN
+F 0 "U4" H 8050 6300 60  0000 C CNN
 F 1 "LM324" H 8150 5900 50  0000 C CNN
 F 2 "" H 8000 6100 60  0000 C CNN
@@
 $EndComp
 $Comp
-L C C201
+L C C1
 U 1 1 523643FC
 P 7250 3950
-F 0 "C201" H 7250 4050 40  0000 L CNN
+F 0 "C1" H 7250 4050 40  0000 L CNN
 F 1 "C" H 7256 3865 40  0000 L CNN
 F 2 "~" H 7288 3800 30  0000 C CNN
@@
 $EndComp
 $Comp
-L R R205
+L R R11
 U 1 1 5236440B
 P 8100 2750
-F 0 "R205" V 8180 2750 40  0000 C CNN
+F 0 "R11" V 8180 2750 40  0000 C CNN
 F 1 "R" V 8107 2751 40  0000 C CNN
 F 2 "~" V 8030 2750 30  0000 C CNN
@@
 $EndComp
 $Comp
-L R R206
+L R R12
 U 1 1 52364427
 P 8100 3400
-F 0 "R206" V 8180 3400 40  0000 C CNN
+F 0 "R12" V 8180 3400 40  0000 C CNN
 F 1 "R" V 8107 3401 40  0000 C CNN
 F 2 "~" V 8030 3400 30  0000 C CNN
@@
 $EndComp
 $Comp
-L R R207
+L R R13
 U 1 1 5236442D
 P 8100 4000
-F 0 "R207" V 8180 4000 40  0000 C CNN
+F 0 "R13" V 8180 4000 40  0000 C CNN
 F 1 "R" V 8107 4001 40  0000 C CNN
 F 2 "~" V 8030 4000 30  0000 C CNN
@@
 $EndComp
 $Comp
-L R R203
+L R R9
 U 1 1 5236444F
 P 7300 2350
-F 0 "R203" V 7380 2350 40  0000 C CNN
+F 0 "R9" V 7380 2350 40  0000 C CNN
 F 1 "R" V 7307 2351 40  0000 C CNN
 F 2 "~" V 7230 2350 30  0000 C CNN
@@
 $EndComp
 $Comp
-L R R202
+L R R8
 U 1 1 52364455
 P 5400 2350
-F 0 "R202" V 5480 2350 40  0000 C CNN
+F 0 "R8" V 5480 2350 40  0000 C CNN
 F 1 "R" V 5407 2351 40  0000 C CNN
 F 2 "~" V 5330 2350 30  0000 C CNN
@@
 $EndComp
 $Comp
-L R R201
+L R R7
 U 1 1 5236445B
 P 5350 4450
-F 0 "R201" V 5430 4450 40  0000 C CNN
+F 0 "R7" V 5430 4450 40  0000 C CNN
 F 1 "R" V 5357 4451 40  0000 C CNN
 F 2 "~" V 5280 4450 30  0000 C CNN
@@
 $EndComp
 $Comp
-L R R204
+L R R10
 U 1 1 52364461
 P 7300 4450
-F 0 "R204" V 7380 4450 40  0000 C CNN
+F 0 "R10" V 7380 4450 40  0000 C CNN
 F 1 "R" V 7307 4451 40  0000 C CNN
 F 2 "~" V 7230 4450 30  0000 C CNN
@@
 $EndComp
 $Comp
-L -12V #PWR01
+L -12V #PWR3
 U 1 1 523646A5
 P 6250 2800
-F 0 "#PWR01" H 6250 2930 20  0001 C CNN
+F 0 "#PWR3" H 6250 2930 20  0001 C CNN
 F 1 "-12V" H 6250 2900 30  0000 C CNN
 F 2 "" H 6250 2800 60  0000 C CNN
@@
 $EndComp
 $Comp
-L -12V #PWR02
+L -12V #PWR6
 U 1 1 523646B2
 P 9000 2850
-F 0 "#PWR02" H 9000 2980 20  0001 C CNN
+F 0 "#PWR6" H 9000 2980 20  0001 C CNN
 F 1 "-12V" H 9000 2950 30  0000 C CNN
 F 2 "" H 9000 2850 60  0000 C CNN
@@
 $EndComp
 $Comp
-L -12V #PWR03
+L -12V #PWR7
 U 1 1 523646B8
 P 9000 3950
-F 0 "#PWR03" H 9000 4080 20  0001 C CNN
+F 0 "#PWR7" H 9000 4080 20  0001 C CNN
 F 1 "-12V" H 9000 4050 30  0000 C CNN
 F 2 "" H 9000 3950 60  0000 C CNN
@@
 $EndComp
 $Comp
-L +12V #PWR04
+L +12V #PWR4
 U 1 1 5236471D
 P 6250 3850
-F 0 "#PWR04" H 6250 3800 20  0001 C CNN
+F 0 "#PWR4" H 6250 3800 20  0001 C CNN
 F 1 "+12V" H 6250 3950 30  0000 C CNN
 F 2 "" H 6250 3850 60  0000 C CNN
@@
 $EndComp
 $Comp
-L +12V #PWR05
+L +12V #PWR5
 U 1 1 5236474B
 P 9000 1800
-F 0 "#PWR05" H 9000 1750 20  0001 C CNN
+F 0 "#PWR5" H 9000 1750 20  0001 C CNN
 F 1 "+12V" H 9000 1900 30  0000 C CNN
 F 2 "" H 9000 1800 60  0000 C CNN
@@
 $EndComp
 $Comp
-L +12V #PWR06
+L +12V #PWR8
 U 1 1 52364796
 P 9000 5000
-F 0 "#PWR06" H 9000 4950 20  0001 C CNN
+F 0 "#PWR8" H 9000 4950 20  0001 C CNN
 F 1 "+12V" H 9000 5100 30  0000 C CNN
 F 2 "" H 9000 5000 60  0000 C CNN
@@
 	9000 5000 9000 4850
 $Comp
-L AGND #PWR07
+L AGND #PWR2
 U 1 1 52364808
 P 4900 4700
-F 0 "#PWR07" H 4900 4700 40  0001 C CNN
+F 0 "#PWR2" H 4900 4700 40  0001 C CNN
 F 1 "AGND" H 4900 4630 50  0000 C CNN
 F 2 "" H 4900 4700 60  0000 C CNN
@@
 	4900 3600 4900 4700
 $Comp
-L MCP3550-60-E/SN U201
+L MCP3550-60-E/SN U2
 U 1 1 5236486B
 P 2350 3450
-F 0 "U201" H 1800 3800 40  0000 C CNN
+F 0 "U2" H 1800 3800 40  0000 C CNN
 F 1 "MCP3550-60-E/SN" H 2050 3750 40  0000 C CNN
 F 2 "SO8" H 2150 3450 30  0000 C CIN
@@
 	950  3550 1850 3550
 $Comp
-L MCP3550-60-E/SN U202
+L MCP3550-60-E/SN U3
 U 1 1 523649E1
 P 2350 6100
-F 0 "U202" H 1800 6450 40  0000 C CNN
+F 0 "U3" H 1800 6450 40  0000 C CNN
 F 1 "MCP3550-60-E/SN" H 2050 6400 40  0000 C CNN
 F 2 "SO8" H 2150 6100 30  0000 C CIN
@@
 $EndComp
 $Comp
-L ZENER D201
+L ZENER D3
 U 1 1 523649F3
 P 9700 6250
-F 0 "D201" H 9700 6350 50  0000 C CNN
+F 0 "D3" H 9700 6350 50  0000 C CNN
 F 1 "ZENER" H 9700 6150 40  0000 C CNN
 F 2 "~" H 9700 6250 60  0000 C CNN
@@
 $EndComp
 $Comp
-L +12V #PWR08
+L +12V #PWR9
 U 1 1 52364A00
 P 9700 5700
-F 0 "#PWR08" H 9700 5650 20  0001 C CNN
+F 0 "#PWR9" H 9700 5650 20  0001 C CNN
 F 1 "+12V" H 9700 5800 30  0000 C CNN
 F 2 "" H 9700 5700 60  0000 C CNN
@@
 	9700 6450 9700 6700
 $Comp
-L AGND #PWR09
+L AGND #PWR10
 U 1 1 52364A60
 P 9700 6700
-F 0 "#PWR09" H 9700 6700 40  0001 C CNN
+F 0 "#PWR10" H 9700 6700 40  0001 C CNN
 F 1 "AGND" H 9700 6630 50  0000 C CNN
 F 2 "" H 9700 6700 60  0000 C CNN
@@
 Connection ~ 7250 6100
 $Comp
-L AGND #PWR010
+L AGND #PWR1
 U 1 1 52364B5B
 P 3000 6450
-F 0 "#PWR010" H 3000 6450 40  0001 C CNN
+F 0 "#PWR1" H 3000 6450 40  0001 C CNN
 F 1 "AGND" H 3000 6380 50  0000 C CNN
 F 2 "" H 3000 6450 60  0000 C CNN
