File: BenchBudEE/BenchBuddy.kicad_pcb (KiCad board)
At the start: 4 copper layers, 165.1 x 63.5 mm, 0 parts

Commit message: syncing to https://github.com/ContextualElectronics/BenchBudEE/tree/ebd662c68b928f78643cdf924dc35a4d91f03121
Changed lines of the file:
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@@
-(kicad_pcb (version 3) (host pcbnew "(2013-07-07 BZR 4022)-stable")
+(kicad_pcb (version 3) (host pcbnew "(2013-03-19 BZR 4004)-stable")
   (general
     (links 0)
     (no_connects 0)
-    (area 0 0 0 0)
+    (area 136.195999 95.682999 301.446001 159.333001)
     (thickness 1.6)
     (drawings 4)
@@
     (title BenchBudEE)
     (rev A)
-    (company "Pepas Labs")
+    (company "Contextual Electronics")
   )
   (layers
@@
     (trace_min 0.1524)
     (segment_width 0.2)
-    (edge_width 0.1)
+    (edge_width 0.15)
     (via_size 0.889)
     (via_drill 0.635)
@@
     (uvia_min_drill 0.127)
     (pcb_text_width 0.3)
-    (pcb_text_size 1.5 1.5)
+    (pcb_text_size 1 1)
     (mod_edge_width 0.15)
     (mod_text_size 1 1)
     (mod_text_width 0.15)
-    (pad_size 1.5 1.5)
+    (pad_size 1 1)
     (pad_drill 0.6)
     (pad_to_mask_clearance 0.254)
@@
       (usegerberextensions true)
       (excludeedgelayer true)
-      (linewidth 0.150000)
+      (linewidth 152400)
       (plotframeref false)
       (viasonmask false)
@@
     (add_net "")
   )
-  (gr_line (start 68.58 195.58) (end 68.58 259.08) (angle 90) (layer Edge.Cuts) (width 0.1))
-  (gr_line (start 233.68 195.58) (end 68.58 195.58) (angle 90) (layer Edge.Cuts) (width 0.1))
-  (gr_line (start 233.68 259.08) (end 233.68 195.58) (angle 90) (layer Edge.Cuts) (width 0.1))
-  (gr_line (start 68.58 259.08) (end 233.68 259.08) (angle 90) (layer Edge.Cuts) (width 0.1))
+  (gr_line (start 136.271 95.758) (end 136.271 159.258) (angle 90) (layer Edge.Cuts) (width 0.15))
+  (gr_line (start 301.371 95.758) (end 136.271 95.758) (angle 90) (layer Edge.Cuts) (width 0.15))
+  (gr_line (start 301.371 159.258) (end 301.371 95.758) (angle 90) (layer Edge.Cuts) (width 0.15))
+  (gr_line (start 136.271 159.258) (end 301.371 159.258) (angle 90) (layer Edge.Cuts) (width 0.15))
 )

Commit message: playing with the layout
Parts:
- added D1: LG Q971-KN-1, LED-0603, F.Cu at (216.5, 131.4)
- added Q1: 2N3904, SOT23EBC, F.Cu at (207.6, 130.2)
- added R1: 500, SM0805, F.Cu at (219.7, 121.3)
- added R2: 200, SM0805, F.Cu at (216.5, 128.3)
- added R3: 0, SM0805, F.Cu at (209.6, 135.3)
- added R4: 100, SM0805, F.Cu at (212.1, 131.4)
- added R5: 0, SM0805, F.Cu at (214.0, 135.3)
- added R6: 0, SM0805, F.Cu at (212.1, 128.3)
Routing:
- net N-0000090: track 0.00 -> 5.81 mm
- net N-0000089: track 0.00 -> 2.97 mm
- net N-0000091: track 0.00 -> 2.74 mm
- net N-0000085: track 0.00 -> 2.63 mm
- net GND: track 0.00 -> 2.54 mm
- net +12P: track 0.00 -> 2.54 mm

Commit message: syncing to upstream
Parts:
- added D2: B130-13-F, SMA, F.Cu at (259.6, 113.9)
- added K1: 1461069-5, TE-SPDT, F.Cu at (269.6, 105.9)
- added U1: LTV-816S, 4-SMD, F.Cu at (254.8, 98.7)
- Q1, R1, R2, R4, R5, R6: moved to B.Cu
- moved R5 66.7 mm to (269.1, 97.7)
- moved Q1 62.9 mm to (268.1, 112.9), turned to 0 degrees
- moved R6 62.2 mm to (272.8, 114.6)
- moved R3 56.9 mm to (257.6, 104.8), turned to 0 degrees
- moved R4 56.5 mm to (264.0, 109.1), turned to 270 degrees
- moved D1 54.6 mm to (264.2, 104.8), turned to 270 degrees
- moved R2 50.8 mm to (261.6, 104.8), turned to 90 degrees
- moved R1 38.9 mm to (252.3, 100.1), turned to 270 degrees
Routing:
- net N-0000090: track 5.81 -> 0.00 mm
- net N-0000089: track 2.97 -> 0.00 mm
- net N-0000091: track 2.74 -> 0.00 mm
- net N-0000085: track 2.63 -> 0.00 mm
- net GND: track 2.54 -> 0.00 mm
- net +12P: track 2.54 -> 0.00 mm

Commit message: playing around with the routing.
Parts:
- Q1, R1, R2, R4, R5, R6: moved to F.Cu
- moved R6 65.5 mm to (210.8, 135.9), turned to 180 degrees
- moved D1 63.9 mm to (207.0, 133.3), turned to 180 degrees
- moved R2 62.9 mm to (207.0, 135.9), turned to 0 degrees
- moved R1 62.0 mm to (200.0, 133.3), turned to 90 degrees
- moved U1 61.6 mm to (200.0, 127.0)
- moved R5 61.1 mm to (213.4, 122.6), turned to 270 degrees
- moved R4 58.5 mm to (210.8, 133.3), turned to 0 degrees
- moved Q1 57.5 mm to (214.6, 134.0), turned to 90 degrees
- moved K1 54.1 mm to (220.3, 128.3)
- moved D2 49.0 mm to (213.4, 130.2)
- moved R3 46.5 mm to (213.4, 119.4), turned to 180 degrees
Routing:
- net N-0000088: track 0.00 -> 12.3 mm
- net N-0000084: track 0.00 -> 12.0 mm
- net N-0000087: track 0.00 -> 10.7 mm
- net N-0000091: track 0.00 -> 6.26 mm
- net N-0000086: track 0.00 -> 2.86 mm
- net N-0000090: track 0.00 -> 2.62 mm
- net +12P: track 0.00 -> 2.62 mm
- net N-0000089: track 0.00 -> 2.26 mm
- net N-0000085: track 0.00 -> 1.95 mm
- net GND: track 0.00 -> 1.91 mm
